File: PCB/DSP board/MCU_Power.sch (KiCad schematic (older format))
At the start: 42 parts, among them U1 STM32H743II

Commit message: Schematics + Footprints Rev.1
Ready to route.
Parts:
- C10, C11, C12, C13, C14, C16, C17, C18, C19, C20, C21, C22, C23, C24, C25, C26, C27, C28, C29, C30, C31, C32, C33, C34, C35, C36, C37, C38, C39, C40, C41, C42, C43, C44, C6, C7, C8, C9: footprint (none) -> Capacitors_SMD:C_0603
- C15: footprint (none) -> Capacitors_SMD:C_0805
- L1, L2: footprint (none) -> Inductors_SMD:L_0603
- U1: footprint (none) -> Housings_QFP:LQFP-176_24x24mm_Pitch0.5mm

Commit message: Schematics & PCB
Schematics update - ERC error fixing
PCB - setup & PCB outline
Parts:
- renumbered C6 to C301, C7 to C302, C8 to C303, C9 to C304, C10 to C305, C11 to C306, C12 to C307, C13 to C308, C14 to C309, C15 to C310, C16 to C311, C17 to C312, C18 to C313, C19 to C314, C20 to C315, C21 to C316, C22 to C317, C23 to C318, C24 to C319, C25 to C320, C26 to C321, C27 to C322, C28 to C323, C29 to C324, C30 to C325, C31 to C326, C32 to C327, C33 to C328, C34 to C329, C35 to C330, C36 to C331, C37 to C332, C38 to C333, C39 to C334, C40 to C335, C41 to C336, C42 to C337, C43 to C338, C44 to C339, L1 to L301, L2 to L302, U1 to U201

Commit message: Component Placement - RN
All components placed except for RAM Resistor Networks
Parts:
- removed C325: 1uF, Capacitors_SMD:C_0603, symbol C_Small
- removed C328: 10nF, Capacitors_SMD:C_0603, symbol C_Small
Other:
- moved on the sheet: C332, C335
Changed lines of the file:
@@
 $EndComp
 $Comp
-L C_Small C325
-U 1 1 5AADC1D1
+L C_Small C332
+U 1 1 5AADC2BC
 P 3200 1850
-F 0 "C325" H 3210 1920 50  0000 L CNN
+F 0 "C332" H 3210 1920 50  0000 L CNN
 F 1 "1uF" H 3210 1770 50  0000 L CNN
 F 2 "Capacitors_SMD:C_0603" H 3200 1850 50  0001 C CNN
@@
 $EndComp
 $Comp
-L C_Small C328
-U 1 1 5AADC1D7
+L C_Small C335
+U 1 1 5AADC2C2
 P 3475 1850
-F 0 "C328" H 3485 1920 50  0000 L CNN
+F 0 "C335" H 3485 1920 50  0000 L CNN
 F 1 "10nF" H 3485 1770 50  0000 L CNN
 F 2 "Capacitors_SMD:C_0603" H 3475 1850 50  0001 C CNN
 F 3 "" H 3475 1850 50  0001 C CNN
 	1    3475 1850
-	1    0    0    -1
-$EndComp
-$Comp
-L C_Small C332
-U 1 1 5AADC2BC
-P 3775 1850
-F 0 "C332" H 3785 1920 50  0000 L CNN
-F 1 "1uF" H 3785 1770 50  0000 L CNN
-F 2 "Capacitors_SMD:C_0603" H 3775 1850 50  0001 C CNN
-F 3 "" H 3775 1850 50  0001 C CNN
-	1    3775 1850
-	1    0    0    -1
-$EndComp
-$Comp
-L C_Small C335
-U 1 1 5AADC2C2
-P 4050 1850
-F 0 "C335" H 4060 1920 50  0000 L CNN
-F 1 "10nF" H 4060 1770 50  0000 L CNN
-F 2 "Capacitors_SMD:C_0603" H 4050 1850 50  0001 C CNN
-F 3 "" H 4050 1850 50  0001 C CNN
-	1    4050 1850
 	1    0    0    -1
 $EndComp
@@
 Connection ~ 1825 775
 Wire Wire Line
-	1300 1675 4050 1675
-Wire Wire Line
-	4050 1675 4050 1750
-Wire Wire Line
-	3775 1750 3775 1675
-Connection ~ 3775 1675
-Wire Wire Line
-	3475 1750 3475 1675
-Connection ~ 3475 1675
-Wire Wire Line
-	3200 1750 3200 1675
+	3475 1675 3475 1750
+Wire Wire Line
+	3200 1675 3200 1750
 Connection ~ 3200 1675
 Wire Wire Line
-	2875 1750 2875 1675
+	2875 1675 2875 1750
 Connection ~ 2875 1675
 Wire Wire Line
-	2600 1750 2600 1675
+	2600 1675 2600 1750
 Connection ~ 2600 1675
 Wire Wire Line
-	2300 1750 2300 1675
+	2300 1675 2300 1750
 Connection ~ 2300 1675
 Wire Wire Line
-	2025 1750 2025 1675
+	2025 1675 2025 1750
 Connection ~ 2025 1675
 Wire Wire Line
-	1700 1750 1700 1675
+	1700 1675 1700 1750
 Connection ~ 1700 1675
 Wire Wire Line
@@
 	1425 1950 1425 2025
 Wire Wire Line
-	1425 2025 4050 2025
+	1425 2025 3475 2025
 Wire Wire Line
 	2775 2025 2775 2075
-Wire Wire Line
-	4050 2025 4050 1950
 Connection ~ 2775 2025
 Wire Wire Line
-	3775 1950 3775 2025
-Connection ~ 3775 2025
-Wire Wire Line
-	3475 1950 3475 2025
-Connection ~ 3475 2025
+	3475 2025 3475 1950
 Wire Wire Line
 	3200 1950 3200 2025
@@
 Connection ~ 1725 3450
 Wire Wire Line
-	2325 4550 1950 4550
-Wire Wire Line
-	2325 4700 2100 4700
+	1950 4550 2325 4550
+Wire Wire Line
+	2100 4700 2325 4700
 Wire Wire Line
 	2100 4450 2100 6500
@@
 	3525 6350 5075 6350
 Wire Wire Line
-	3700 6350 3700 4550
+	3700 4550 3700 6350
 Wire Wire Line
 	3525 6200 3700 6200
@@
 	1    0    0    -1
 $EndComp
+Wire Wire Line
+	1300 1675 3475 1675
 $EndSCHEMATC
