File: PCB/DSP board/Main board.sch (KiCad schematic (older format))
At the start: 5 parts, among them X101 Mini_PCI-e

Commit message: Added Testpoints
Parts:
- added TP101, TP102, TP103, TP104, TP105, TP106, TP107, TP108, TP109, TP110, TP111: TEST, Measurement_Points:Measurement_Point_Round-SMD-Pad_Small, symbol TEST
Connections:
- net GND: now also TP109.1
- new net +3V3: TP104.1
- new net +3V3_LDO: TP106.1
- new net +5V: TP105.1
- new net D+: TP110.1
- new net D-: TP111.1
- new net NRST: TP103.1
- new net PROG_CLK: TP101.1
- new net PROG_IO: TP102.1
- new net TFT_LED+: TP107.1
- new net TFT_LED-: TP108.1
Changed lines of the file:
@@
 NoConn ~ 6575 4900
 $Comp
-L PWR_FLAG #FLG07
+L PWR_FLAG #FLG06
 U 1 1 5ABDE685
 P 9750 3800
-F 0 "#FLG07" H 9750 3875 50  0001 C CNN
+F 0 "#FLG06" H 9750 3875 50  0001 C CNN
 F 1 "PWR_FLAG" H 9750 3950 50  0000 C CNN
 F 2 "" H 9750 3800 50  0001 C CNN
@@
 Text GLabel 9825 3875 2    60   Input ~ 0
 +3V3_MCU
+$Comp
+L TEST TP101
+U 1 1 5AC72D8A
+P 7700 5100
+F 0 "TP101" H 7700 5400 50  0000 C BNN
+F 1 "TEST" H 7700 5350 50  0000 C CNN
+F 2 "Measurement_Points:Measurement_Point_Round-SMD-Pad_Small" H 7700 5100 50  0001 C CNN
+F 3 "" H 7700 5100 50  0001 C CNN
+	1    7700 5100
+	1    0    0    -1
+$EndComp
+$Comp
+L TEST TP102
+U 1 1 5AC72EF3
+P 7950 5100
+F 0 "TP102" H 7950 5400 50  0000 C BNN
+F 1 "TEST" H 7950 5350 50  0000 C CNN
+F 2 "Measurement_Points:Measurement_Point_Round-SMD-Pad_Small" H 7950 5100 50  0001 C CNN
+F 3 "" H 7950 5100 50  0001 C CNN
+	1    7950 5100
+	1    0    0    -1
+$EndComp
+$Comp
+L TEST TP103
+U 1 1 5AC72F20
+P 8200 5100
+F 0 "TP103" H 8200 5400 50  0000 C BNN
+F 1 "TEST" H 8200 5350 50  0000 C CNN
+F 2 "Measurement_Points:Measurement_Point_Round-SMD-Pad_Small" H 8200 5100 50  0001 C CNN
+F 3 "" H 8200 5100 50  0001 C CNN
+	1    8200 5100
+	1    0    0    -1
+$EndComp
+$Comp
+L TEST TP104
+U 1 1 5AC72F47
+P 8575 5100
+F 0 "TP104" H 8575 5400 50  0000 C BNN
+F 1 "TEST" H 8575 5350 50  0000 C CNN
+F 2 "Measurement_Points:Measurement_Point_Round-SMD-Pad_Small" H 8575 5100 50  0001 C CNN
+F 3 "" H 8575 5100 50  0001 C CNN
+	1    8575 5100
+	1    0    0    -1
+$EndComp
+$Comp
+L TEST TP105
+U 1 1 5AC72F70
+P 8825 5100
+F 0 "TP105" H 8825 5400 50  0000 C BNN
+F 1 "TEST" H 8825 5350 50  0000 C CNN
+F 2 "Measurement_Points:Measurement_Point_Round-SMD-Pad_Small" H 8825 5100 50  0001 C CNN
+F 3 "" H 8825 5100 50  0001 C CNN
+	1    8825 5100
+	1    0    0    -1
+$EndComp
+$Comp
+L TEST TP106
+U 1 1 5AC72F9B
+P 9100 5100
+F 0 "TP106" H 9100 5400 50  0000 C BNN
+F 1 "TEST" H 9100 5350 50  0000 C CNN
+F 2 "Measurement_Points:Measurement_Point_Round-SMD-Pad_Small" H 9100 5100 50  0001 C CNN
+F 3 "" H 9100 5100 50  0001 C CNN
+	1    9100 5100
+	1    0    0    -1
+$EndComp
+$Comp
+L TEST TP107
+U 1 1 5AC73010
+P 9475 5100
+F 0 "TP107" H 9475 5400 50  0000 C BNN
+F 1 "TEST" H 9475 5350 50  0000 C CNN
+F 2 "Measurement_Points:Measurement_Point_Round-SMD-Pad_Small" H 9475 5100 50  0001 C CNN
+F 3 "" H 9475 5100 50  0001 C CNN
+	1    9475 5100
+	1    0    0    -1
+$EndComp
+$Comp
+L TEST TP108
+U 1 1 5AC7304D
+P 9725 5100
+F 0 "TP108" H 9725 5400 50  0000 C BNN
+F 1 "TEST" H 9725 5350 50  0000 C CNN
+F 2 "Measurement_Points:Measurement_Point_Round-SMD-Pad_Small" H 9725 5100 50  0001 C CNN
+F 3 "" H 9725 5100 50  0001 C CNN
+	1    9725 5100
+	1    0    0    -1
+$EndComp
+$Comp
+L TEST TP109
+U 1 1 5AC730B1
+P 10250 5075
+F 0 "TP109" H 10250 5375 50  0000 C BNN
+F 1 "TEST" H 10250 5325 50  0000 C CNN
+F 2 "Measurement_Points:Measurement_Point_Round-SMD-Pad_Small" H 10250 5075 50  0001 C CNN
+F 3 "" H 10250 5075 50  0001 C CNN
+	1    10250 5075
+	1    0    0    -1
+$EndComp
+Text GLabel 7700 5225 3    60   Output ~ 0
+PROG_CLK
+Text GLabel 7950 5225 3    60   BiDi ~ 0
+PROG_IO
+Text GLabel 8200 5225 3    60   BiDi ~ 0
+NRST
+$Comp
+L GND #PWR07
+U 1 1 5AC74D7E
+P 10250 5125
+F 0 "#PWR07" H 10250 4875 50  0001 C CNN
+F 1 "GND" V 10250 4850 50  0000 C CNN
+F 2 "" H 10250 5125 50  0001 C CNN
+F 3 "" H 10250 5125 50  0001 C CNN
+	1    10250 5125
+	1    0    0    -1
+$EndComp
+Wire Wire Line
+	10250 5075 10250 5125
+Wire Wire Line
+	7700 5100 7700 5225
+Wire Wire Line
+	7950 5100 7950 5225
+Wire Wire Line
+	8200 5100 8200 5225
+$Comp
+L +3V3 #PWR08
+U 1 1 5AC75E25
+P 8575 5250
+F 0 "#PWR08" H 8575 5100 50  0001 C CNN
+F 1 "+3V3" H 8575 5390 50  0000 C CNN
+F 2 "" H 8575 5250 50  0001 C CNN
+F 3 "" H 8575 5250 50  0001 C CNN
+	1    8575 5250
+	-1   0    0    1
+$EndComp
+Wire Wire Line
+	8575 5250 8575 5100
+$Comp
+L +5V #PWR09
+U 1 1 5AC75ED2
+P 8825 5250
+F 0 "#PWR09" H 8825 5100 50  0001 C CNN
+F 1 "+5V" H 8825 5390 50  0000 C CNN
+F 2 "" H 8825 5250 50  0001 C CNN
+F 3 "" H 8825 5250 50  0001 C CNN
+	1    8825 5250
+	-1   0    0    1
+$EndComp
+Wire Wire Line
+	8825 5100 8825 5250
+Text GLabel 9100 5225 3    60   Input ~ 0
++3V3_LDO
+Wire Wire Line
+	9100 5100 9100 5225
+Text GLabel 9475 5225 3    60   Input ~ 0
+TFT_LED+
+Text GLabel 9725 5225 3    60   Input ~ 0
+TFT_LED-
+Wire Wire Line
+	9475 5225 9475 5100
+Wire Wire Line
+	9725 5100 9725 5225
+$Comp
+L TEST TP110
+U 1 1 5AC78159
+P 10550 5075
+F 0 "TP110" H 10550 5375 50  0000 C BNN
+F 1 "TEST" H 10550 5325 50  0000 C CNN
+F 2 "Measurement_Points:Measurement_Point_Round-SMD-Pad_Small" H 10550 5075 50  0001 C CNN
+F 3 "" H 10550 5075 50  0001 C CNN
+	1    10550 5075
+	1    0    0    -1
+$EndComp
+$Comp
+L TEST TP111
+U 1 1 5AC781D5
+P 10800 5075
+F 0 "TP111" H 10800 5375 50  0000 C BNN
+F 1 "TEST" H 10800 5325 50  0000 C CNN
+F 2 "Measurement_Points:Measurement_Point_Round-SMD-Pad_Small" H 10800 5075 50  0001 C CNN
+F 3 "" H 10800 5075 50  0001 C CNN
+	1    10800 5075
+	1    0    0    -1
+$EndComp
+Text GLabel 10550 5150 3    60   BiDi ~ 0
+D+
+Text GLabel 10800 5150 3    60   BiDi ~ 0
+D-
+Wire Wire Line
+	10550 5150 10550 5075
+Wire Wire Line
+	10800 5150 10800 5075
 $EndSCHEMATC
