File: PCB/DSP board/RAM.sch (KiCad schematic (older format))
At the start: 27 parts, among them U2 AS4C32M8SA

Commit message: Schematics + Footprints Rev.1
Ready to route.
Parts:
- C45, C46, C48, C49, C50, C51, C52, C53, C54, C55, C56, C57, C58, C59, C60, C61: footprint (none) -> Capacitors_SMD:C_0603
- C47: footprint (none) -> Capacitors_SMD:C_0805
- L3: footprint (none) -> Inductors_SMD:L_0603
- RN10, RN3, RN4, RN5, RN6, RN7, RN8, RN9: footprint (none) -> Resistor:0603_RN4
- U2: footprint (none) -> TSSOP:TSSOP-54_P-0.8mm
Connections:
- net FMC__SDNCAS renamed FMC_SDNCAS
Changed lines of the file:
@@
 F 0 "U2" H 3550 3725 60  0000 C CNN
 F 1 "AS4C32M8SA" H 3600 575 60  0000 C CNN
-F 2 "" H 3550 3725 60  0001 C CNN
+F 2 "TSSOP:TSSOP-54_P-0.8mm" H 3550 3725 60  0001 C CNN
 F 3 "" H 3550 3725 60  0001 C CNN
 	1    3650 2175
@@
 F 0 "U2" H 3550 7525 60  0000 C CNN
 F 1 "AS4C32M8SA" H 3600 4375 60  0000 C CNN
-F 2 "" H 3550 7525 60  0001 C CNN
+F 2 "TSSOP:TSSOP-54_P-0.8mm" H 3550 7525 60  0001 C CNN
 F 3 "" H 3550 7525 60  0001 C CNN
 	2    3650 5975
@@
 F 0 "U2" H 8950 5400 60  0000 C CNN
 F 1 "AS4C32M8SA" H 9000 2250 60  0000 C CNN
-F 2 "" H 8950 5400 60  0001 C CNN
+F 2 "TSSOP:TSSOP-54_P-0.8mm" H 8950 5400 60  0001 C CNN
 F 3 "" H 8950 5400 60  0001 C CNN
 	3    9050 3850
@@
 $EndComp
 $Comp
-L +3V3 #PWR28
+L +3V3 #PWR028
 U 1 1 5AB09085
 P 4425 675
-F 0 "#PWR28" H 4425 525 50  0001 C CNN
+F 0 "#PWR028" H 4425 525 50  0001 C CNN
 F 1 "+3V3" V 4500 850 50  0000 C CNN
 F 2 "" H 4425 675 50  0001 C CNN
@@
 F 0 "L3" V 5225 725 50  0000 L CNN
 F 1 "220R" V 5000 500 50  0000 L CNN
-F 2 "" V 5055 675 50  0001 C CNN
+F 2 "Inductors_SMD:L_0603" V 5055 675 50  0001 C CNN
 F 3 "" H 5125 675 50  0001 C CNN
 	1    5125 675
@@
 F 0 "C45" H 4560 895 50  0000 L CNN
 F 1 "1uF" H 4560 745 50  0000 L CNN
-F 2 "" H 4550 825 50  0001 C CNN
+F 2 "Capacitors_SMD:C_0603" H 4550 825 50  0001 C CNN
 F 3 "" H 4550 825 50  0001 C CNN
 	1    4550 825
@@
 F 0 "C46" H 4810 895 50  0000 L CNN
 F 1 "10nF" H 4810 745 50  0000 L CNN
-F 2 "" H 4800 825 50  0001 C CNN
+F 2 "Capacitors_SMD:C_0603" H 4800 825 50  0001 C CNN
 F 3 "" H 4800 825 50  0001 C CNN
 	1    4800 825
@@
 $EndComp
 $Comp
-L GND #PWR29
+L GND #PWR029
 U 1 1 5AB09981
 P 4550 975
-F 0 "#PWR29" H 4550 725 50  0001 C CNN
+F 0 "#PWR029" H 4550 725 50  0001 C CNN
 F 1 "GND" H 4550 825 50  0000 C CNN
 F 2 "" H 4550 975 50  0001 C CNN
@@
 $EndComp
 $Comp
-L GND #PWR30
+L GND #PWR030
 U 1 1 5AB099A1
 P 4800 975
-F 0 "#PWR30" H 4800 725 50  0001 C CNN
+F 0 "#PWR030" H 4800 725 50  0001 C CNN
 F 1 "GND" H 4800 825 50  0000 C CNN
 F 2 "" H 4800 975 50  0001 C CNN
@@
 F 0 "C47" H 5485 895 50  0000 L CNN
 F 1 "4.7uF" H 5485 745 50  0000 L CNN
-F 2 "" H 5475 825 50  0001 C CNN
+F 2 "Capacitors_SMD:C_0805" H 5475 825 50  0001 C CNN
 F 3 "" H 5475 825 50  0001 C CNN
 	1    5475 825
@@
 $EndComp
 $Comp
-L GND #PWR31
+L GND #PWR031
 U 1 1 5AB09D89
 P 5475 975
-F 0 "#PWR31" H 5475 725 50  0001 C CNN
+F 0 "#PWR031" H 5475 725 50  0001 C CNN
 F 1 "GND" H 5475 825 50  0000 C CNN
 F 2 "" H 5475 975 50  0001 C CNN
@@
 F 0 "C48" H 7135 920 50  0000 L CNN
 F 1 "1uF" H 7135 770 50  0000 L CNN
-F 2 "" H 7125 850 50  0001 C CNN
+F 2 "Capacitors_SMD:C_0603" H 7125 850 50  0001 C CNN
 F 3 "" H 7125 850 50  0001 C CNN
 	1    7125 850
@@
 F 0 "C49" H 7410 920 50  0000 L CNN
 F 1 "10nF" H 7410 770 50  0000 L CNN
-F 2 "" H 7400 850 50  0001 C CNN
+F 2 "Capacitors_SMD:C_0603" H 7400 850 50  0001 C CNN
 F 3 "" H 7400 850 50  0001 C CNN
 	1    7400 850
@@
 F 0 "C50" H 7735 920 50  0000 L CNN
 F 1 "1uF" H 7735 770 50  0000 L CNN
-F 2 "" H 7725 850 50  0001 C CNN
+F 2 "Capacitors_SMD:C_0603" H 7725 850 50  0001 C CNN
 F 3 "" H 7725 850 50  0001 C CNN
 	1    7725 850
@@
 F 0 "C51" H 8010 920 50  0000 L CNN
 F 1 "10nF" H 8010 770 50  0000 L CNN
-F 2 "" H 8000 850 50  0001 C CNN
+F 2 "Capacitors_SMD:C_0603" H 8000 850 50  0001 C CNN
 F 3 "" H 8000 850 50  0001 C CNN
 	1    8000 850
@@
 F 0 "C52" H 8310 920 50  0000 L CNN
 F 1 "1uF" H 8310 770 50  0000 L CNN
-F 2 "" H 8300 850 50  0001 C CNN
+F 2 "Capacitors_SMD:C_0603" H 8300 850 50  0001 C CNN
 F 3 "" H 8300 850 50  0001 C CNN
 	1    8300 850
@@
 F 0 "C53" H 8585 920 50  0000 L CNN
 F 1 "10nF" H 8585 770 50  0000 L CNN
-F 2 "" H 8575 850 50  0001 C CNN
+F 2 "Capacitors_SMD:C_0603" H 8575 850 50  0001 C CNN
 F 3 "" H 8575 850 50  0001 C CNN
 	1    8575 850
@@
 F 0 "C54" H 8910 920 50  0000 L CNN
 F 1 "1uF" H 8910 770 50  0000 L CNN
-F 2 "" H 8900 850 50  0001 C CNN
+F 2 "Capacitors_SMD:C_0603" H 8900 850 50  0001 C CNN
 F 3 "" H 8900 850 50  0001 C CNN
 	1    8900 850
@@
 F 0 "C55" H 9210 920 50  0000 L CNN
 F 1 "10nF" H 9210 770 50  0000 L CNN
-F 2 "" H 9200 850 50  0001 C CNN
+F 2 "Capacitors_SMD:C_0603" H 9200 850 50  0001 C CNN
 F 3 "" H 9200 850 50  0001 C CNN
 	1    9200 850
@@
 F 0 "C56" H 9510 920 50  0000 L CNN
 F 1 "1uF" H 9510 770 50  0000 L CNN
-F 2 "" H 9500 850 50  0001 C CNN
+F 2 "Capacitors_SMD:C_0603" H 9500 850 50  0001 C CNN
 F 3 "" H 9500 850 50  0001 C CNN
 	1    9500 850
@@
 F 0 "C57" H 9785 920 50  0000 L CNN
 F 1 "10nF" H 9785 770 50  0000 L CNN
-F 2 "" H 9775 850 50  0001 C CNN
+F 2 "Capacitors_SMD:C_0603" H 9775 850 50  0001 C CNN
 F 3 "" H 9775 850 50  0001 C CNN
 	1    9775 850
@@
 $EndComp
 $Comp
-L GND #PWR33
+L GND #PWR032
 U 1 1 5AB0D087
 P 9050 1100
-F 0 "#PWR33" H 9050 850 50  0001 C CNN
+F 0 "#PWR032" H 9050 850 50  0001 C CNN
 F 1 "GND" H 9050 950 50  0000 C CNN
 F 2 "" H 9050 1100 50  0001 C CNN
@@
 F 0 "C58" H 10085 920 50  0000 L CNN
 F 1 "1uF" H 10085 770 50  0000 L CNN
-F 2 "" H 10075 850 50  0001 C CNN
+F 2 "Capacitors_SMD:C_0603" H 10075 850 50  0001 C CNN
 F 3 "" H 10075 850 50  0001 C CNN
 	1    10075 850
@@
 F 0 "C59" H 10360 920 50  0000 L CNN
 F 1 "10nF" H 10360 770 50  0000 L CNN
-F 2 "" H 10350 850 50  0001 C CNN
+F 2 "Capacitors_SMD:C_0603" H 10350 850 50  0001 C CNN
 F 3 "" H 10350 850 50  0001 C CNN
 	1    10350 850
@@
 F 0 "C60" H 10660 920 50  0000 L CNN
 F 1 "1uF" H 10660 770 50  0000 L CNN
-F 2 "" H 10650 850 50  0001 C CNN
+F 2 "Capacitors_SMD:C_0603" H 10650 850 50  0001 C CNN
 F 3 "" H 10650 850 50  0001 C CNN
 	1    10650 850
@@
 F 0 "C61" H 10935 920 50  0000 L CNN
 F 1 "10nF" H 10935 770 50  0000 L CNN
-F 2 "" H 10925 850 50  0001 C CNN
+F 2 "Capacitors_SMD:C_0603" H 10925 850 50  0001 C CNN
 F 3 "" H 10925 850 50  0001 C CNN
 	1    10925 850
@@
 F 0 "RN3" V 1325 975 50  0000 C CNN
 F 1 "51R" V 1825 975 50  0000 C CNN
-F 2 "" V 1900 975 50  0001 C CNN
+F 2 "Resistor:0603_RN4" V 1900 975 50  0001 C CNN
 F 3 "" H 1625 975 50  0001 C CNN
 	1    1625 975
@@
 F 0 "RN4" V 1325 1800 50  0000 C CNN
 F 1 "51R" V 1825 1800 50  0000 C CNN
-F 2 "" V 1900 1800 50  0001 C CNN
+F 2 "Resistor:0603_RN4" V 1900 1800 50  0001 C CNN
 F 3 "" H 1625 1800 50  0001 C CNN
 	1    1625 1800
@@
 F 0 "RN5" V 1325 2625 50  0000 C CNN
 F 1 "51R" V 1825 2625 50  0000 C CNN
-F 2 "" V 1900 2625 50  0001 C CNN
+F 2 "Resistor:0603_RN4" V 1900 2625 50  0001 C CNN
 F 3 "" H 1625 2625 50  0001 C CNN
 	1    1625 2625
@@
 F 0 "RN6" V 1325 3500 50  0000 C CNN
 F 1 "51R" V 1825 3500 50  0000 C CNN
-F 2 "" V 1900 3500 50  0001 C CNN
+F 2 "Resistor:0603_RN4" V 1900 3500 50  0001 C CNN
 F 3 "" H 1625 3500 50  0001 C CNN
 	1    1625 3500
@@
 F 0 "RN7" V 1325 4750 50  0000 C CNN
 F 1 "51R" V 1825 4750 50  0000 C CNN
-F 2 "" V 1900 4750 50  0001 C CNN
+F 2 "Resistor:0603_RN4" V 1900 4750 50  0001 C CNN
 F 3 "" H 1625 4750 50  0001 C CNN
 	1    1625 4750
@@
 F 0 "RN8" V 1325 5575 50  0000 C CNN
 F 1 "51R" V 1825 5575 50  0000 C CNN
-F 2 "" V 1900 5575 50  0001 C CNN
+F 2 "Resistor:0603_RN4" V 1900 5575 50  0001 C CNN
 F 3 "" H 1625 5575 50  0001 C CNN
 	1    1625 5575
@@
 F 0 "RN9" V 1325 6400 50  0000 C CNN
 F 1 "51R" V 1825 6400 50  0000 C CNN
-F 2 "" V 1900 6400 50  0001 C CNN
+F 2 "Resistor:0603_RN4" V 1900 6400 50  0001 C CNN
 F 3 "" H 1625 6400 50  0001 C CNN
 	1    1625 6400
@@
 F 0 "RN10" V 1325 7275 50  0000 C CNN
 F 1 "51R" V 1825 7275 50  0000 C CNN
-F 2 "" V 1900 7275 50  0001 C CNN
+F 2 "Resistor:0603_RN4" V 1900 7275 50  0001 C CNN
 F 3 "" H 1625 7275 50  0001 C CNN
 	1    1625 7275
@@
 FMC_SDNWE
 Text GLabel 1325 1700 0    60   Input ~ 0
-FMC__SDNCAS
+FMC_SDNCAS
 Text GLabel 1325 1800 0    60   Input ~ 0
 FMC_SDNRAS
@@
 	8450 3650 8450 2450
 $Comp
-L GND #PWR32
+L GND #PWR033
 U 1 1 5AB60DC8
 P 8450 5200
-F 0 "#PWR32" H 8450 4950 50  0001 C CNN
+F 0 "#PWR033" H 8450 4950 50  0001 C CNN
 F 1 "GND" H 8450 5050 50  0000 C CNN
 F 2 "" H 8450 5200 50  0001 C CNN

Commit message: Schematics & PCB
Schematics update - ERC error fixing
PCB - setup & PCB outline
Parts:
- renumbered C45 to C401, C46 to C402, C47 to C403, C48 to C404, C49 to C405, C50 to C406, C51 to C407, C52 to C408, C53 to C409, C54 to C410, C55 to C411, C56 to C412, C57 to C413, C58 to C414, C59 to C415, C60 to C416, C61 to C417, L3 to L401, RN3 to RN401, RN4 to RN402, RN5 to RN403, RN6 to RN404, RN7 to RN405, RN8 to RN406, RN9 to RN407, RN10 to RN408, U2 to U401
Connections:
- no-connect marks 0 -> 4
Changed lines of the file:
@@
 $EndDescr
 $Comp
-L AS4C32M8SA U2
+L AS4C32M8SA U401
 U 1 1 5AB086F2
 P 3650 2175
-F 0 "U2" H 3550 3725 60  0000 C CNN
+F 0 "U401" H 3550 3725 60  0000 C CNN
 F 1 "AS4C32M8SA" H 3600 575 60  0000 C CNN
 F 2 "TSSOP:TSSOP-54_P-0.8mm" H 3550 3725 60  0001 C CNN
@@
 $EndComp
 $Comp
-L AS4C32M8SA U2
+L AS4C32M8SA U401
 U 2 1 5AB0884F
 P 3650 5975
-F 0 "U2" H 3550 7525 60  0000 C CNN
+F 0 "U401" H 3550 7525 60  0000 C CNN
 F 1 "AS4C32M8SA" H 3600 4375 60  0000 C CNN
 F 2 "TSSOP:TSSOP-54_P-0.8mm" H 3550 7525 60  0001 C CNN
@@
 $EndComp
 $Comp
-L AS4C32M8SA U2
+L AS4C32M8SA U401
 U 3 1 5AB088F8
 P 9050 3850
-F 0 "U2" H 8950 5400 60  0000 C CNN
+F 0 "U401" H 8950 5400 60  0000 C CNN
 F 1 "AS4C32M8SA" H 9000 2250 60  0000 C CNN
 F 2 "TSSOP:TSSOP-54_P-0.8mm" H 8950 5400 60  0001 C CNN
@@
 $EndComp
 $Comp
-L +3V3 #PWR028
+L +3V3 #PWR031
 U 1 1 5AB09085
 P 4425 675
-F 0 "#PWR028" H 4425 525 50  0001 C CNN
+F 0 "#PWR031" H 4425 525 50  0001 C CNN
 F 1 "+3V3" V 4500 850 50  0000 C CNN
 F 2 "" H 4425 675 50  0001 C CNN
@@
 $EndComp
 $Comp
-L Ferrite_Bead_Small L3
+L Ferrite_Bead_Small L401
 U 1 1 5AB09469
 P 5125 675
-F 0 "L3" V 5225 725 50  0000 L CNN
+F 0 "L401" V 5225 725 50  0000 L CNN
 F 1 "220R" V 5000 500 50  0000 L CNN
 F 2 "Inductors_SMD:L_0603" V 5055 675 50  0001 C CNN
@@
 $EndComp
 $Comp
-L C_Small C45
+L C_Small C401
 U 1 1 5AB098BA
 P 4550 825
-F 0 "C45" H 4560 895 50  0000 L CNN
+F 0 "C401" H 4560 895 50  0000 L CNN
 F 1 "1uF" H 4560 745 50  0000 L CNN
 F 2 "Capacitors_SMD:C_0603" H 4550 825 50  0001 C CNN
@@
 $EndComp
 $Comp
-L C_Small C46
+L C_Small C402
 U 1 1 5AB0990E
 P 4800 825
-F 0 "C46" H 4810 895 50  0000 L CNN
+F 0 "C402" H 4810 895 50  0000 L CNN
 F 1 "10nF" H 4810 745 50  0000 L CNN
 F 2 "Capacitors_SMD:C_0603" H 4800 825 50  0001 C CNN
@@
 $EndComp
 $Comp
-L GND #PWR029
+L GND #PWR032
 U 1 1 5AB09981
 P 4550 975
-F 0 "#PWR029" H 4550 725 50  0001 C CNN
+F 0 "#PWR032" H 4550 725 50  0001 C CNN
 F 1 "GND" H 4550 825 50  0000 C CNN
 F 2 "" H 4550 975 50  0001 C CNN
@@
 $EndComp
 $Comp
-L GND #PWR030
+L GND #PWR033
 U 1 1 5AB099A1
 P 4800 975
-F 0 "#PWR030" H 4800 725 50  0001 C CNN
+F 0 "#PWR033" H 4800 725 50  0001 C CNN
 F 1 "GND" H 4800 825 50  0000 C CNN
 F 2 "" H 4800 975 50  0001 C CNN
@@
 $EndComp
 $Comp
-L C_Small C47
+L C_Small C403
 U 1 1 5AB09CA1
 P 5475 825
-F 0 "C47" H 5485 895 50  0000 L CNN
+F 0 "C403" H 5485 895 50  0000 L CNN
 F 1 "4.7uF" H 5485 745 50  0000 L CNN
 F 2 "Capacitors_SMD:C_0805" H 5475 825 50  0001 C CNN
@@
 $EndComp
 $Comp
-L GND #PWR031
+L GND #PWR034
 U 1 1 5AB09D89
 P 5475 975
-F 0 "#PWR031" H 5475 725 50  0001 C CNN
+F 0 "#PWR034" H 5475 725 50  0001 C CNN
 F 1 "GND" H 5475 825 50  0000 C CNN
 F 2 "" H 5475 975 50  0001 C CNN
@@
 +3V3_RAM
 $Comp
-L C_Small C48
+L C_Small C404
 U 1 1 5AB0D041
 P 7125 850
-F 0 "C48" H 7135 920 50  0000 L CNN
+F 0 "C404" H 7135 920 50  0000 L CNN
 F 1 "1uF" H 7135 770 50  0000 L CNN
 F 2 "Capacitors_SMD:C_0603" H 7125 850 50  0001 C CNN
@@
 $EndComp
 $Comp
-L C_Small C49
+L C_Small C405
 U 1 1 5AB0D048
 P 7400 850
-F 0 "C49" H 7410 920 50  0000 L CNN
+F 0 "C405" H 7410 920 50  0000 L CNN
 F 1 "10nF" H 7410 770 50  0000 L CNN
 F 2 "Capacitors_SMD:C_0603" H 7400 850 50  0001 C CNN
@@
 $EndComp
 $Comp
-L C_Small C50
+L C_Small C406
 U 1 1 5AB0D04F
 P 7725 850
-F 0 "C50" H 7735 920 50  0000 L CNN
+F 0 "C406" H 7735 920 50  0000 L CNN
 F 1 "1uF" H 7735 770 50  0000 L CNN
 F 2 "Capacitors_SMD:C_0603" H 7725 850 50  0001 C CNN
@@
 $EndComp
 $Comp
-L C_Small C51
+L C_Small C407
 U 1 1 5AB0D056
 P 8000 850
-F 0 "C51" H 8010 920 50  0000 L CNN
+F 0 "C407" H 8010 920 50  0000 L CNN
 F 1 "10nF" H 8010 770 50  0000 L CNN
 F 2 "Capacitors_SMD:C_0603" H 8000 850 50  0001 C CNN
@@
 $EndComp
 $Comp
-L C_Small C52
+L C_Small C408
 U 1 1 5AB0D05D
 P 8300 850
-F 0 "C52" H 8310 920 50  0000 L CNN
+F 0 "C408" H 8310 920 50  0000 L CNN
 F 1 "1uF" H 8310 770 50  0000 L CNN
 F 2 "Capacitors_SMD:C_0603" H 8300 850 50  0001 C CNN
@@
 $EndComp
 $Comp
-L C_Small C53
+L C_Small C409
 U 1 1 5AB0D064
 P 8575 850
-F 0 "C53" H 8585 920 50  0000 L CNN
+F 0 "C409" H 8585 920 50  0000 L CNN
 F 1 "10nF" H 8585 770 50  0000 L CNN
 F 2 "Capacitors_SMD:C_0603" H 8575 850 50  0001 C CNN
@@
 $EndComp
 $Comp
-L C_Small C54
+L C_Small C410
 U 1 1 5AB0D06B
 P 8900 850
-F 0 "C54" H 8910 920 50  0000 L CNN
+F 0 "C410" H 8910 920 50  0000 L CNN
 F 1 "1uF" H 8910 770 50  0000 L CNN
 F 2 "Capacitors_SMD:C_0603" H 8900 850 50  0001 C CNN
@@
 $EndComp
 $Comp
-L C_Small C55
+L C_Small C411
 U 1 1 5AB0D072
 P 9200 850
-F 0 "C55" H 9210 920 50  0000 L CNN
+F 0 "C411" H 9210 920 50  0000 L CNN
 F 1 "10nF" H 9210 770 50  0000 L CNN
 F 2 "Capacitors_SMD:C_0603" H 9200 850 50  0001 C CNN
@@
 $EndComp
 $Comp
-L C_Small C56
+L C_Small C412
 U 1 1 5AB0D079
 P 9500 850
-F 0 "C56" H 9510 920 50  0000 L CNN
+F 0 "C412" H 9510 920 50  0000 L CNN
 F 1 "1uF" H 9510 770 50  0000 L CNN
 F 2 "Capacitors_SMD:C_0603" H 9500 850 50  0001 C CNN
@@
 $EndComp
 $Comp
-L C_Small C57
+L C_Small C413
 U 1 1 5AB0D080
 P 9775 850
-F 0 "C57" H 9785 920 50  0000 L CNN
+F 0 "C413" H 9785 920 50  0000 L CNN
 F 1 "10nF" H 9785 770 50  0000 L CNN
 F 2 "Capacitors_SMD:C_0603" H 9775 850 50  0001 C CNN
@@
 $EndComp
 $Comp
-L GND #PWR032
+L GND #PWR035
 U 1 1 5AB0D087
 P 9050 1100
-F 0 "#PWR032" H 9050 850 50  0001 C CNN
+F 0 "#PWR035" H 9050 850 50  0001 C CNN
 F 1 "GND" H 9050 950 50  0000 C CNN
 F 2 "" H 9050 1100 50  0001 C CNN
@@
 Connection ~ 7400 1025
 $Comp
-L C_Small C58
+L C_Small C414
 U 1 1 5AB0E0F3
 P 10075 850
-F 0 "C58" H 10085 920 50  0000 L CNN
+F 0 "C414" H 10085 920 50  0000 L CNN
 F 1 "1uF" H 10085 770 50  0000 L CNN
 F 2 "Capacitors_SMD:C_0603" H 10075 850 50  0001 C CNN
@@
 $EndComp
 $Comp
-L C_Small C59
+L C_Small C415
 U 1 1 5AB0E0F9
 P 10350 850
-F 0 "C59" H 10360 920 50  0000 L CNN
+F 0 "C415" H 10360 920 50  0000 L CNN
 F 1 "10nF" H 10360 770 50  0000 L CNN
 F 2 "Capacitors_SMD:C_0603" H 10350 850 50  0001 C CNN
@@
 $EndComp
 $Comp
-L C_Small C60
+L C_Small C416
 U 1 1 5AB0E0FF
 P 10650 850
-F 0 "C60" H 10660 920 50  0000 L CNN
+F 0 "C416" H 10660 920 50  0000 L CNN
 F 1 "1uF" H 10660 770 50  0000 L CNN
 F 2 "Capacitors_SMD:C_0603" H 10650 850 50  0001 C CNN
@@
 $EndComp
 $Comp
-L C_Small C61
+L C_Small C417
 U 1 1 5AB0E105
 P 10925 850
-F 0 "C61" H 10935 920 50  0000 L CNN
+F 0 "C417" H 10935 920 50  0000 L CNN
 F 1 "10nF" H 10935 770 50  0000 L CNN
 F 2 "Capacitors_SMD:C_0603" H 10925 850 50  0001 C CNN
@@
 Connection ~ 9050 1025
 $Comp
-L R_Pack04 RN3
+L R_Pack04 RN401
 U 1 1 5AB111FD
 P 1625 975
-F 0 "RN3" V 1325 975 50  0000 C CNN
+F 0 "RN401" V 1325 975 50  0000 C CNN
 F 1 "51R" V 1825 975 50  0000 C CNN
 F 2 "Resistor:0603_RN4" V 1900 975 50  0001 C CNN
@@
 $EndComp
 $Comp
-L R_Pack04 RN4
+L R_Pack04 RN402
 U 1 1 5AB11920
 P 1625 1800
-F 0 "RN4" V 1325 1800 50  0000 C CNN
+F 0 "RN402" V 1325 1800 50  0000 C CNN
 F 1 "51R" V 1825 1800 50  0000 C CNN
 F 2 "Resistor:0603_RN4" V 1900 1800 50  0001 C CNN
@@
 $EndComp
 $Comp
-L R_Pack04 RN5
+L R_Pack04 RN403
 U 1 1 5AB119DD
 P 1625 2625
-F 0 "RN5" V 1325 2625 50  0000 C CNN
+F 0 "RN403" V 1325 2625 50  0000 C CNN
 F 1 "51R" V 1825 2625 50  0000 C CNN
 F 2 "Resistor:0603_RN4" V 1900 2625 50  0001 C CNN
@@
 $EndComp
 $Comp
-L R_Pack04 RN6
+L R_Pack04 RN404
 U 1 1 5AB11A42
 P 1625 3500
-F 0 "RN6" V 1325 3500 50  0000 C CNN
+F 0 "RN404" V 1325 3500 50  0000 C CNN
 F 1 "51R" V 1825 3500 50  0000 C CNN
 F 2 "Resistor:0603_RN4" V 1900 3500 50  0001 C CNN
@@
 $EndComp
 $Comp
-L R_Pack04 RN7
+L R_Pack04 RN405
 U 1 1 5AB18C9F
 P 1625 4750
-F 0 "RN7" V 1325 4750 50  0000 C CNN
+F 0 "RN405" V 1325 4750 50  0000 C CNN
 F 1 "51R" V 1825 4750 50  0000 C CNN
 F 2 "Resistor:0603_RN4" V 1900 4750 50  0001 C CNN
@@
 $EndComp
 $Comp
-L R_Pack04 RN8
+L R_Pack04 RN406
 U 1 1 5AB18CA5
 P 1625 5575
-F 0 "RN8" V 1325 5575 50  0000 C CNN
+F 0 "RN406" V 1325 5575 50  0000 C CNN
 F 1 "51R" V 1825 5575 50  0000 C CNN
 F 2 "Resistor:0603_RN4" V 1900 5575 50  0001 C CNN
@@
 $EndComp
 $Comp
-L R_Pack04 RN9
+L R_Pack04 RN407
 U 1 1 5AB18CAB
 P 1625 6400
-F 0 "RN9" V 1325 6400 50  0000 C CNN
+F 0 "RN407" V 1325 6400 50  0000 C CNN
 F 1 "51R" V 1825 6400 50  0000 C CNN
 F 2 "Resistor:0603_RN4" V 1900 6400 50  0001 C CNN
@@
 $EndComp
 $Comp
-L R_Pack04 RN10
+L R_Pack04 RN408
 U 1 1 5AB18CB1
 P 1625 7275
-F 0 "RN10" V 1325 7275 50  0000 C CNN
+F 0 "RN408" V 1325 7275 50  0000 C CNN
 F 1 "51R" V 1825 7275 50  0000 C CNN
 F 2 "Resistor:0603_RN4" V 1900 7275 50  0001 C CNN
@@
 Connection ~ 8450 3650
 Wire Wire Line
-	8450 3650 8450 2450
-$Comp
-L GND #PWR033
+	8450 2350 8450 3650
+$Comp
+L GND #PWR036
 U 1 1 5AB60DC8
 P 8450 5200
-F 0 "#PWR033" H 8450 4950 50  0001 C CNN
+F 0 "#PWR036" H 8450 4950 50  0001 C CNN
 F 1 "GND" H 8450 5050 50  0000 C CNN
 F 2 "" H 8450 5200 50  0001 C CNN
@@
 Text Notes 10300 7500 0    60   ~ 0
 By Jesse Spiessens
+NoConn ~ 1425 4550
+NoConn ~ 1825 4550
+NoConn ~ 1425 3600
+NoConn ~ 1825 3600
+$Comp
+L PWR_FLAG #FLG037
+U 1 1 5ABDFBF6
+P 8450 2350
+F 0 "#FLG037" H 8450 2425 50  0001 C CNN
+F 1 "PWR_FLAG" H 8450 2500 50  0000 C CNN
+F 2 "" H 8450 2350 50  0001 C CNN
+F 3 "" H 8450 2350 50  0001 C CNN
+	1    8450 2350
+	1    0    0    -1
+$EndComp
 $EndSCHEMATC
