File: PCB/DSP board/RAM.sch (KiCad schematic (older format))
At the start: 27 parts, among them U401 AS4C32M8SA

Commit message: RAM Routing - Data
All RAM routing & matching done, supply still needs to be done
Parts:
- removed RN401, RN402, RN403, RN404, RN405, RN406, RN407, RN408: 51R, Resistor:0603_RN4, symbol R_Pack04
Connections:
- net RAM_A0 is gone; now on net FMC_A0: U401.23 (A0)
- net RAM_A1 is gone; now on net FMC_A1: U401.24 (A1)
- net RAM_A10 is gone; now on net FMC_A10: U401.22 (A10)
- net RAM_A11 is gone; now on net FMC_A11: U401.35 (A11)
- net RAM_A12 is gone; now on net FMC_A12: U401.36 (A12)
- net RAM_A2 is gone; now on net FMC_A2: U401.25 (A2)
- net RAM_A3 is gone; now on net FMC_A3: U401.26 (A3)
- net RAM_A4 is gone; now on net FMC_A4: U401.29 (A4)
- net RAM_A5 is gone; now on net FMC_A5: U401.30 (A5)
- net RAM_A6 is gone; now on net FMC_A6: U401.31 (A6)
- net RAM_A7 is gone; now on net FMC_A7: U401.32 (A7)
- net RAM_A8 is gone; now on net FMC_A8: U401.33 (A8)
- net RAM_A9 is gone; now on net FMC_A9: U401.34 (A9)
- net RAM_BA0 is gone; now on net FMC_BA0: U401.20 (BA0)
- net RAM_BA1 is gone; now on net FMC_BA1: U401.21 (BA1)
- net RAM_CAS# is gone; now on net FMC_SDNCAS: U401.17 (CAS#)
- net RAM_CKE is gone; now on net FMC_SDCKE0: U401.37 (CKE)
- net RAM_CLK is gone; now on net FMC_SDCLK: U401.38 (CLK)
- net RAM_CS# is gone; now on net FMC_SDNE0: U401.19 (CS#)
- net RAM_DQ0 is gone; now on net FMC_D0: U401.2 (DQ0)
- net RAM_DQ1 is gone; now on net FMC_D1: U401.5 (DQ1)
- net RAM_DQ2 is gone; now on net FMC_D2: U401.8 (DQ2)
- net RAM_DQ3 is gone; now on net FMC_D3: U401.11 (DQ3)
- net RAM_DQ4 is gone; now on net FMC_D4: U401.44 (DQ4)
- net RAM_DQ5 is gone; now on net FMC_D5: U401.47 (DQ5)
- net RAM_DQ6 is gone; now on net FMC_D6: U401.50 (DQ6)
- net RAM_DQ7 is gone; now on net FMC_D7: U401.53 (DQ7)
- net RAM_DQM is gone; now on net FMC_NBL0: U401.39 (DQM)
- net RAM_RAS# is gone; now on net FMC_SDNRAS: U401.18 (RAS#)
- net RAM_WE# is gone; now on net FMC_SDNWE: U401.16 (WE#)
- no-connect marks 4 -> 0
Changed lines of the file:
@@
 	9050 1100 9050 1025
 Connection ~ 9050 1025
-$Comp
-L R_Pack04 RN401
-U 1 1 5AB111FD
-P 1625 975
-F 0 "RN401" V 1325 975 50  0000 C CNN
-F 1 "51R" V 1825 975 50  0000 C CNN
-F 2 "Resistor:0603_RN4" V 1900 975 50  0001 C CNN
-F 3 "" H 1625 975 50  0001 C CNN
-	1    1625 975
-	0    1    1    0
-$EndComp
-$Comp
-L R_Pack04 RN402
-U 1 1 5AB11920
-P 1625 1800
-F 0 "RN402" V 1325 1800 50  0000 C CNN
-F 1 "51R" V 1825 1800 50  0000 C CNN
-F 2 "Resistor:0603_RN4" V 1900 1800 50  0001 C CNN
-F 3 "" H 1625 1800 50  0001 C CNN
-	1    1625 1800
-	0    1    1    0
-$EndComp
-$Comp
-L R_Pack04 RN403
-U 1 1 5AB119DD
-P 1625 2625
-F 0 "RN403" V 1325 2625 50  0000 C CNN
-F 1 "51R" V 1825 2625 50  0000 C CNN
-F 2 "Resistor:0603_RN4" V 1900 2625 50  0001 C CNN
-F 3 "" H 1625 2625 50  0001 C CNN
-	1    1625 2625
-	0    1    1    0
-$EndComp
-$Comp
-L R_Pack04 RN404
-U 1 1 5AB11A42
-P 1625 3500
-F 0 "RN404" V 1325 3500 50  0000 C CNN
-F 1 "51R" V 1825 3500 50  0000 C CNN
-F 2 "Resistor:0603_RN4" V 1900 3500 50  0001 C CNN
-F 3 "" H 1625 3500 50  0001 C CNN
-	1    1625 3500
-	0    1    1    0
-$EndComp
-$Comp
-L R_Pack04 RN405
-U 1 1 5AB18C9F
-P 1625 4750
-F 0 "RN405" V 1325 4750 50  0000 C CNN
-F 1 "51R" V 1825 4750 50  0000 C CNN
-F 2 "Resistor:0603_RN4" V 1900 4750 50  0001 C CNN
-F 3 "" H 1625 4750 50  0001 C CNN
-	1    1625 4750
-	0    1    1    0
-$EndComp
-$Comp
-L R_Pack04 RN406
-U 1 1 5AB18CA5
-P 1625 5575
-F 0 "RN406" V 1325 5575 50  0000 C CNN
-F 1 "51R" V 1825 5575 50  0000 C CNN
-F 2 "Resistor:0603_RN4" V 1900 5575 50  0001 C CNN
-F 3 "" H 1625 5575 50  0001 C CNN
-	1    1625 5575
-	0    1    1    0
-$EndComp
-$Comp
-L R_Pack04 RN407
-U 1 1 5AB18CAB
-P 1625 6400
-F 0 "RN407" V 1325 6400 50  0000 C CNN
-F 1 "51R" V 1825 6400 50  0000 C CNN
-F 2 "Resistor:0603_RN4" V 1900 6400 50  0001 C CNN
-F 3 "" H 1625 6400 50  0001 C CNN
-	1    1625 6400
-	0    1    1    0
-$EndComp
-$Comp
-L R_Pack04 RN408
-U 1 1 5AB18CB1
-P 1625 7275
-F 0 "RN408" V 1325 7275 50  0000 C CNN
-F 1 "51R" V 1825 7275 50  0000 C CNN
-F 2 "Resistor:0603_RN4" V 1900 7275 50  0001 C CNN
-F 3 "" H 1625 7275 50  0001 C CNN
-	1    1625 7275
-	0    1    1    0
-$EndComp
 Text GLabel 1325 775  0    60   BiDi ~ 0
 FMC_D0
@@
 FMC_A7
 Wire Wire Line
-	1275 7375 1425 7375
-Wire Wire Line
-	1425 7275 1275 7275
-Wire Wire Line
-	1425 7175 1275 7175
-Wire Wire Line
-	1275 7075 1425 7075
-Wire Wire Line
-	1425 6500 1325 6500
-Wire Wire Line
-	1325 6400 1425 6400
-Wire Wire Line
-	1425 6300 1325 6300
-Wire Wire Line
-	1325 6200 1425 6200
-Wire Wire Line
-	1325 5675 1425 5675
-Wire Wire Line
-	1325 5575 1425 5575
-Wire Wire Line
-	1325 5475 1425 5475
-Wire Wire Line
-	1325 5375 1425 5375
-Wire Wire Line
-	1325 4850 1425 4850
-Wire Wire Line
-	1325 4750 1425 4750
-Wire Wire Line
-	1325 4650 1425 4650
-Wire Wire Line
-	1325 3500 1425 3500
-Wire Wire Line
-	1325 3400 1425 3400
-Wire Wire Line
-	1325 3300 1425 3300
-Wire Wire Line
-	1325 2725 1425 2725
-Wire Wire Line
-	1425 2625 1325 2625
-Wire Wire Line
-	1325 2525 1425 2525
-Wire Wire Line
-	1425 2425 1325 2425
-Wire Wire Line
-	1325 1900 1425 1900
-Wire Wire Line
-	1325 1800 1425 1800
-Wire Wire Line
-	1325 1700 1425 1700
-Wire Wire Line
-	1325 1600 1425 1600
-Wire Wire Line
-	1325 1075 1425 1075
-Wire Wire Line
-	1325 975  1425 975
-Wire Wire Line
-	1325 875  1425 875
-Wire Wire Line
-	1325 775  1425 775
+	1275 7375 1925 7375
+Wire Wire Line
+	1275 7275 1925 7275
+Wire Wire Line
+	1275 7175 1925 7175
+Wire Wire Line
+	1275 7075 1925 7075
+Wire Wire Line
+	1325 6500 1925 6500
+Wire Wire Line
+	1325 6400 1925 6400
+Wire Wire Line
+	1325 6300 1925 6300
+Wire Wire Line
+	1325 6200 1925 6200
+Wire Wire Line
+	1325 5675 1925 5675
+Wire Wire Line
+	1325 5575 1925 5575
+Wire Wire Line
+	1325 5475 1925 5475
+Wire Wire Line
+	1325 5375 1925 5375
+Wire Wire Line
+	1325 4850 1925 4850
+Wire Wire Line
+	1325 4750 1925 4750
+Wire Wire Line
+	1325 4650 1925 4650
+Wire Wire Line
+	1325 3500 1925 3500
+Wire Wire Line
+	1325 3400 1925 3400
+Wire Wire Line
+	1325 3300 1925 3300
+Wire Wire Line
+	1325 2725 1925 2725
+Wire Wire Line
+	1325 2625 1925 2625
+Wire Wire Line
+	1325 2525 1925 2525
+Wire Wire Line
+	1325 2425 1925 2425
+Wire Wire Line
+	1325 1900 1925 1900
+Wire Wire Line
+	1325 1800 1925 1800
+Wire Wire Line
+	1325 1700 1925 1700
+Wire Wire Line
+	1325 1600 1925 1600
+Wire Wire Line
+	1325 1075 1925 1075
+Wire Wire Line
+	1325 975  1925 975
+Wire Wire Line
+	1325 875  1925 875
+Wire Wire Line
+	1325 775  1925 775
 Text GLabel 1925 775  2    60   BiDi ~ 0
 RAM_DQ0
@@
 Text GLabel 1925 7375 2    60   BiDi ~ 0
 RAM_DQ7
-Wire Wire Line
-	1825 775  1925 775
-Wire Wire Line
-	1825 875  1925 875
-Wire Wire Line
-	1825 975  1925 975
-Wire Wire Line
-	1925 1075 1825 1075
-Wire Wire Line
-	1825 1600 1925 1600
-Wire Wire Line
-	1925 1700 1825 1700
-Wire Wire Line
-	1825 1800 1925 1800
-Wire Wire Line
-	1925 1900 1825 1900
-Wire Wire Line
-	1825 2425 1925 2425
-Wire Wire Line
-	1925 2525 1825 2525
-Wire Wire Line
-	1825 2625 1925 2625
-Wire Wire Line
-	1925 2725 1825 2725
-Wire Wire Line
-	1825 3300 1925 3300
-Wire Wire Line
-	1925 3400 1825 3400
-Wire Wire Line
-	1825 3500 1925 3500
-Wire Wire Line
-	1825 4650 1925 4650
-Wire Wire Line
-	1925 4750 1825 4750
-Wire Wire Line
-	1825 4850 1925 4850
-Wire Wire Line
-	1825 5375 1925 5375
-Wire Wire Line
-	1925 5475 1825 5475
-Wire Wire Line
-	1825 5575 1925 5575
-Wire Wire Line
-	1925 5675 1825 5675
-Wire Wire Line
-	1825 6200 1925 6200
-Wire Wire Line
-	1925 6300 1825 6300
-Wire Wire Line
-	1825 6400 1925 6400
-Wire Wire Line
-	1925 6500 1825 6500
-Wire Wire Line
-	1825 7075 1925 7075
-Wire Wire Line
-	1925 7175 1825 7175
-Wire Wire Line
-	1825 7275 1925 7275
-Wire Wire Line
-	1925 7375 1825 7375
 Text GLabel 3150 4575 0    60   BiDi ~ 0
 RAM_DQ0
@@
 Text Notes 10300 7500 0    60   ~ 0
 By Jesse Spiessens
-NoConn ~ 1425 4550
-NoConn ~ 1825 4550
-NoConn ~ 1425 3600
-NoConn ~ 1825 3600
 $Comp
 L PWR_FLAG #FLG037
