File: PCB/DSP board/Screen.sch (KiCad schematic (older format))
At the start: 20 parts, among them J2 Conn_01x40_Female, J3 Conn_01x06_Female

Commit message: Schematics + Footprints Rev.1
Ready to route.
Parts:
- C100, C98: footprint (none) -> Capacitors_SMD:C_0603
- C99: footprint (none) -> Capacitors_SMD:C_0805
- D10, D6, D7, D8, D9: footprint (none) -> ESD:U-DFN3810-9
- J2: footprint (none) -> Molex:78127-1408
- J3: footprint (none) -> Molex:52808-0671
- L10: footprint (none) -> Inductors_SMD:L_0603
- RN13, RN14, RN15, RN16, RN17, RN18, RN19, RN20, RN21: footprint (none) -> Resistor:0603_RN4
Changed lines of the file:
@@
 F 0 "J2" H 6225 5525 50  0000 C CNN
 F 1 "Conn_01x40_Female" H 6225 1425 50  0000 C CNN
-F 2 "" H 6225 3525 50  0001 C CNN
+F 2 "Molex:78127-1408" H 6225 3525 50  0001 C CNN
 F 3 "" H 6225 3525 50  0001 C CNN
 	1    6225 3525
@@
 TFT_DEN
 $Comp
-L GND #PWR93
+L GND #PWR083
 U 1 1 5AB957CE
 P 5925 5325
-F 0 "#PWR93" H 5925 5075 50  0001 C CNN
+F 0 "#PWR083" H 5925 5075 50  0001 C CNN
 F 1 "GND" V 5925 5125 50  0000 C CNN
 F 2 "" H 5925 5325 50  0001 C CNN
@@
 $EndComp
 $Comp
-L GND #PWR92
+L GND #PWR084
 U 1 1 5AB9582D
 P 5925 2725
-F 0 "#PWR92" H 5925 2475 50  0001 C CNN
+F 0 "#PWR084" H 5925 2475 50  0001 C CNN
 F 1 "GND" V 5925 2525 50  0000 C CNN
 F 2 "" H 5925 2725 50  0001 C CNN
@@
 $EndComp
 $Comp
-L GND #PWR91
+L GND #PWR085
 U 1 1 5AB9584B
 P 5925 2025
-F 0 "#PWR91" H 5925 1775 50  0001 C CNN
+F 0 "#PWR085" H 5925 1775 50  0001 C CNN
 F 1 "GND" V 5925 1825 50  0000 C CNN
 F 2 "" H 5925 2025 50  0001 C CNN
@@
 	5925 5525 6025 5525
 $Comp
-L +3V3 #PWR83
+L +3V3 #PWR086
 U 1 1 5AB9671A
 P 900 775
-F 0 "#PWR83" H 900 625 50  0001 C CNN
+F 0 "#PWR086" H 900 625 50  0001 C CNN
 F 1 "+3V3" V 925 975 50  0000 C CNN
 F 2 "" H 900 775 50  0001 C CNN
@@
 F 0 "L10" V 1450 825 50  0000 L CNN
 F 1 "220R" V 1225 625 50  0000 L CNN
-F 2 "" V 1280 775 50  0001 C CNN
+F 2 "Inductors_SMD:L_0603" V 1280 775 50  0001 C CNN
 F 3 "" H 1350 775 50  0001 C CNN
 	1    1350 775
@@
 F 0 "C98" H 1085 1020 50  0000 L CNN
 F 1 "10nF" H 1085 870 50  0000 L CNN
-F 2 "" H 1075 950 50  0001 C CNN
+F 2 "Capacitors_SMD:C_0603" H 1075 950 50  0001 C CNN
 F 3 "" H 1075 950 50  0001 C CNN
 	1    1075 950
@@
 F 0 "C99" H 1635 1020 50  0000 L CNN
 F 1 "4.7uF" H 1635 870 50  0000 L CNN
-F 2 "" H 1625 950 50  0001 C CNN
+F 2 "Capacitors_SMD:C_0805" H 1625 950 50  0001 C CNN
 F 3 "" H 1625 950 50  0001 C CNN
 	1    1625 950
@@
 F 0 "C100" H 1960 1020 50  0000 L CNN
 F 1 "10nF" H 1960 870 50  0000 L CNN
-F 2 "" H 1950 950 50  0001 C CNN
+F 2 "Capacitors_SMD:C_0603" H 1950 950 50  0001 C CNN
 F 3 "" H 1950 950 50  0001 C CNN
 	1    1950 950
@@
 $EndComp
 $Comp
-L GND #PWR84
+L GND #PWR087
 U 1 1 5AB9699B
 P 1075 1125
-F 0 "#PWR84" H 1075 875 50  0001 C CNN
+F 0 "#PWR087" H 1075 875 50  0001 C CNN
 F 1 "GND" H 1075 975 50  0000 C CNN
 F 2 "" H 1075 1125 50  0001 C CNN
@@
 $EndComp
 $Comp
-L GND #PWR85
+L GND #PWR088
 U 1 1 5AB969B9
 P 1625 1125
-F 0 "#PWR85" H 1625 875 50  0001 C CNN
+F 0 "#PWR088" H 1625 875 50  0001 C CNN
 F 1 "GND" H 1625 975 50  0000 C CNN
 F 2 "" H 1625 1125 50  0001 C CNN
@@
 $EndComp
 $Comp
-L GND #PWR86
+L GND #PWR089
 U 1 1 5AB969D7
 P 1950 1125
-F 0 "#PWR86" H 1950 875 50  0001 C CNN
+F 0 "#PWR089" H 1950 875 50  0001 C CNN
 F 1 "GND" H 1950 975 50  0000 C CNN
 F 2 "" H 1950 1125 50  0001 C CNN
@@
 F 0 "RN14" V 1600 2625 50  0000 C CNN
 F 1 "51R" V 2100 2625 50  0000 C CNN
-F 2 "" V 2175 2625 50  0001 C CNN
+F 2 "Resistor:0603_RN4" V 2175 2625 50  0001 C CNN
 F 3 "" H 1900 2625 50  0001 C CNN
 	1    1900 2625
@@
 F 0 "RN15" V 1600 3400 50  0000 C CNN
 F 1 "51R" V 2100 3400 50  0000 C CNN
-F 2 "" V 2175 3400 50  0001 C CNN
+F 2 "Resistor:0603_RN4" V 2175 3400 50  0001 C CNN
 F 3 "" H 1900 3400 50  0001 C CNN
 	1    1900 3400
@@
 F 0 "RN16" V 1600 4175 50  0000 C CNN
 F 1 "51R" V 2100 4175 50  0000 C CNN
-F 2 "" V 2175 4175 50  0001 C CNN
+F 2 "Resistor:0603_RN4" V 2175 4175 50  0001 C CNN
 F 3 "" H 1900 4175 50  0001 C CNN
 	1    1900 4175
@@
 F 0 "RN17" V 1600 4950 50  0000 C CNN
 F 1 "51R" V 2100 4950 50  0000 C CNN
-F 2 "" V 2175 4950 50  0001 C CNN
+F 2 "Resistor:0603_RN4" V 2175 4950 50  0001 C CNN
 F 3 "" H 1900 4950 50  0001 C CNN
 	1    1900 4950
@@
 F 0 "RN18" V 1600 5750 50  0000 C CNN
 F 1 "51R" V 2100 5750 50  0000 C CNN
-F 2 "" V 2175 5750 50  0001 C CNN
+F 2 "Resistor:0603_RN4" V 2175 5750 50  0001 C CNN
 F 3 "" H 1900 5750 50  0001 C CNN
 	1    1900 5750
@@
 F 0 "RN19" V 1600 6525 50  0000 C CNN
 F 1 "51R" V 2100 6525 50  0000 C CNN
-F 2 "" V 2175 6525 50  0001 C CNN
+F 2 "Resistor:0603_RN4" V 2175 6525 50  0001 C CNN
 F 3 "" H 1900 6525 50  0001 C CNN
 	1    1900 6525
@@
 F 0 "RN20" V 1600 7300 50  0000 C CNN
 F 1 "51R" V 2100 7300 50  0000 C CNN
-F 2 "" V 2175 7300 50  0001 C CNN
+F 2 "Resistor:0603_RN4" V 2175 7300 50  0001 C CNN
 F 3 "" H 1900 7300 50  0001 C CNN
 	1    1900 7300
@@
 F 0 "RN13" V 1600 1875 50  0000 C CNN
 F 1 "51R" V 2100 1875 50  0000 C CNN
-F 2 "" V 2175 1875 50  0001 C CNN
+F 2 "Resistor:0603_RN4" V 2175 1875 50  0001 C CNN
 F 3 "" H 1900 1875 50  0001 C CNN
 	1    1900 1875
@@
 F 0 "D6" H 4150 2675 60  0000 C CNN
 F 1 "DT1240A-08LP3810" H 4350 1525 60  0000 C CNN
-F 2 "" H 4100 1625 60  0001 C CNN
+F 2 "ESD:U-DFN3810-9" H 4100 1625 60  0001 C CNN
 F 3 "" H 4100 1625 60  0001 C CNN
 	1    4350 2125
@@
 F 0 "D7" H 4150 4200 60  0000 C CNN
 F 1 "DT1240A-08LP3810" H 4350 3050 60  0000 C CNN
-F 2 "" H 4100 3150 60  0001 C CNN
+F 2 "ESD:U-DFN3810-9" H 4100 3150 60  0001 C CNN
 F 3 "" H 4100 3150 60  0001 C CNN
 	1    4350 3650
@@
 F 0 "D8" H 4150 5750 60  0000 C CNN
 F 1 "DT1240A-08LP3810" H 4350 4600 60  0000 C CNN
-F 2 "" H 4100 4700 60  0001 C CNN
+F 2 "ESD:U-DFN3810-9" H 4100 4700 60  0001 C CNN
 F 3 "" H 4100 4700 60  0001 C CNN
 	1    4350 5200
@@
 F 0 "D9" H 4150 7325 60  0000 C CNN
 F 1 "DT1240A-08LP3810" H 4350 6175 60  0000 C CNN
-F 2 "" H 4100 6275 60  0001 C CNN
+F 2 "ESD:U-DFN3810-9" H 4100 6275 60  0001 C CNN
 F 3 "" H 4100 6275 60  0001 C CNN
 	1    4350 6775
@@
 	3800 7175 3900 7175
 $Comp
-L GND #PWR88
+L GND #PWR090
 U 1 1 5ABB29AB
 P 3875 2125
-F 0 "#PWR88" H 3875 1875 50  0001 C CNN
+F 0 "#PWR090" H 3875 1875 50  0001 C CNN
 F 1 "GND" V 3875 1925 50  0000 C CNN
 F 2 "" H 3875 2125 50  0001 C CNN
@@
 	3875 2125 3900 2125
 $Comp
-L GND #PWR89
+L GND #PWR091
 U 1 1 5ABB2CDD
 P 3875 3650
-F 0 "#PWR89" H 3875 3400 50  0001 C CNN
+F 0 "#PWR091" H 3875 3400 50  0001 C CNN
 F 1 "GND" V 3875 3450 50  0000 C CNN
 F 2 "" H 3875 3650 50  0001 C CNN
@@
 $EndComp
 $Comp
-L GND #PWR90
+L GND #PWR092
 U 1 1 5ABB3065
 P 3875 5200
-F 0 "#PWR90" H 3875 4950 50  0001 C CNN
+F 0 "#PWR092" H 3875 4950 50  0001 C CNN
 F 1 "GND" V 3875 5000 50  0000 C CNN
 F 2 "" H 3875 5200 50  0001 C CNN
@@
 $EndComp
 $Comp
-L GND #PWR87
+L GND #PWR093
 U 1 1 5ABB33CB
 P 3850 6775
-F 0 "#PWR87" H 3850 6525 50  0001 C CNN
+F 0 "#PWR093" H 3850 6525 50  0001 C CNN
 F 1 "GND" V 3850 6575 50  0000 C CNN
 F 2 "" H 3850 6775 50  0001 C CNN
@@
 F 0 "J3" H 10400 3600 50  0000 C CNN
 F 1 "Conn_01x06_Female" H 10400 2900 50  0000 C CNN
-F 2 "" H 10400 3300 50  0001 C CNN
+F 2 "Molex:52808-0671" H 10400 3300 50  0001 C CNN
 F 3 "" H 10400 3300 50  0001 C CNN
 	1    10400 3300
@@
 F 0 "D10" H 9925 2550 60  0000 C CNN
 F 1 "DT1240A-08LP3810" H 10125 1400 60  0000 C CNN
-F 2 "" H 9875 1500 60  0001 C CNN
+F 2 "ESD:U-DFN3810-9" H 9875 1500 60  0001 C CNN
 F 3 "" H 9875 1500 60  0001 C CNN
 	1    10125 2000
@@
 TFT_SCL
 $Comp
-L GND #PWR95
+L GND #PWR094
 U 1 1 5ABC279B
 P 10150 3500
-F 0 "#PWR95" H 10150 3250 50  0001 C CNN
+F 0 "#PWR094" H 10150 3250 50  0001 C CNN
 F 1 "GND" V 10150 3300 50  0000 C CNN
 F 2 "" H 10150 3500 50  0001 C CNN
@@
 Connection ~ 9600 2350
 $Comp
-L GND #PWR94
+L GND #PWR095
 U 1 1 5ABC535D
 P 9600 2000
-F 0 "#PWR94" H 9600 1750 50  0001 C CNN
+F 0 "#PWR095" H 9600 1750 50  0001 C CNN
 F 1 "GND" V 9600 1800 50  0000 C CNN
 F 2 "" H 9600 2000 50  0001 C CNN
@@
 F 0 "RN21" V 7500 1850 50  0000 C CNN
 F 1 "51R" V 8000 1850 50  0000 C CNN
-F 2 "" V 8075 1850 50  0001 C CNN
+F 2 "Resistor:0603_RN4" V 8075 1850 50  0001 C CNN
 F 3 "" H 7800 1850 50  0001 C CNN
 	1    7800 1850

Commit message: Schematics & PCB
Schematics update - ERC error fixing
PCB - setup & PCB outline
Parts:
- renumbered C98 to C701, C99 to C702, C100 to C703, D6 to D701, D7 to D702, D8 to D703, D9 to D704, D10 to D705, J2 to J701, J3 to J702, L10 to L701, RN13 to RN701, RN14 to RN702, RN15 to RN703, RN16 to RN704, RN17 to RN705, RN18 to RN706, RN19 to RN707, RN20 to RN708, RN21 to RN709
Connections:
- no-connect marks 0 -> 17
Changed lines of the file:
@@
 $EndDescr
 $Comp
-L Conn_01x40_Female J2
+L Conn_01x40_Female J701
 U 1 1 5AB94CC4
 P 6225 3525
-F 0 "J2" H 6225 5525 50  0000 C CNN
+F 0 "J701" H 6225 5525 50  0000 C CNN
 F 1 "Conn_01x40_Female" H 6225 1425 50  0000 C CNN
 F 2 "Molex:78127-1408" H 6225 3525 50  0001 C CNN
@@
 TFT_DEN
 $Comp
-L GND #PWR083
+L GND #PWR093
 U 1 1 5AB957CE
 P 5925 5325
-F 0 "#PWR083" H 5925 5075 50  0001 C CNN
+F 0 "#PWR093" H 5925 5075 50  0001 C CNN
 F 1 "GND" V 5925 5125 50  0000 C CNN
 F 2 "" H 5925 5325 50  0001 C CNN
@@
 $EndComp
 $Comp
-L GND #PWR084
+L GND #PWR094
 U 1 1 5AB9582D
 P 5925 2725
-F 0 "#PWR084" H 5925 2475 50  0001 C CNN
+F 0 "#PWR094" H 5925 2475 50  0001 C CNN
 F 1 "GND" V 5925 2525 50  0000 C CNN
 F 2 "" H 5925 2725 50  0001 C CNN
@@
 $EndComp
 $Comp
-L GND #PWR085
+L GND #PWR095
 U 1 1 5AB9584B
 P 5925 2025
-F 0 "#PWR085" H 5925 1775 50  0001 C CNN
+F 0 "#PWR095" H 5925 1775 50  0001 C CNN
 F 1 "GND" V 5925 1825 50  0000 C CNN
 F 2 "" H 5925 2025 50  0001 C CNN
@@
 	5925 5525 6025 5525
 $Comp
-L +3V3 #PWR086
+L +3V3 #PWR096
 U 1 1 5AB9671A
 P 900 775
-F 0 "#PWR086" H 900 625 50  0001 C CNN
+F 0 "#PWR096" H 900 625 50  0001 C CNN
 F 1 "+3V3" V 925 975 50  0000 C CNN
 F 2 "" H 900 775 50  0001 C CNN
@@
 $EndComp
 $Comp
-L Ferrite_Bead_Small L10
+L Ferrite_Bead_Small L701
 U 1 1 5AB9678B
 P 1350 775
-F 0 "L10" V 1450 825 50  0000 L CNN
+F 0 "L701" V 1450 825 50  0000 L CNN
 F 1 "220R" V 1225 625 50  0000 L CNN
 F 2 "Inductors_SMD:L_0603" V 1280 775 50  0001 C CNN
@@
 $EndComp
 $Comp
-L C_Small C98
+L C_Small C701
 U 1 1 5AB967F0
 P 1075 950
-F 0 "C98" H 1085 1020 50  0000 L CNN
+F 0 "C701" H 1085 1020 50  0000 L CNN
 F 1 "10nF" H 1085 870 50  0000 L CNN
 F 2 "Capacitors_SMD:C_0603" H 1075 950 50  0001 C CNN
@@
 $EndComp
 $Comp
-L C_Small C99
+L C_Small C702
 U 1 1 5AB9683F
 P 1625 950
-F 0 "C99" H 1635 1020 50  0000 L CNN
+F 0 "C702" H 1635 1020 50  0000 L CNN
 F 1 "4.7uF" H 1635 870 50  0000 L CNN
 F 2 "Capacitors_SMD:C_0805" H 1625 950 50  0001 C CNN
@@
 $EndComp
 $Comp
-L C_Small C100
+L C_Small C703
 U 1 1 5AB96876
 P 1950 950
-F 0 "C100" H 1960 1020 50  0000 L CNN
+F 0 "C703" H 1960 1020 50  0000 L CNN
 F 1 "10nF" H 1960 870 50  0000 L CNN
 F 2 "Capacitors_SMD:C_0603" H 1950 950 50  0001 C CNN
@@
 $EndComp
 $Comp
-L GND #PWR087
+L GND #PWR097
 U 1 1 5AB9699B
 P 1075 1125
-F 0 "#PWR087" H 1075 875 50  0001 C CNN
+F 0 "#PWR097" H 1075 875 50  0001 C CNN
 F 1 "GND" H 1075 975 50  0000 C CNN
 F 2 "" H 1075 1125 50  0001 C CNN
@@
 $EndComp
 $Comp
-L GND #PWR088
+L GND #PWR098
 U 1 1 5AB969B9
 P 1625 1125
-F 0 "#PWR088" H 1625 875 50  0001 C CNN
+F 0 "#PWR098" H 1625 875 50  0001 C CNN
 F 1 "GND" H 1625 975 50  0000 C CNN
 F 2 "" H 1625 1125 50  0001 C CNN
@@
 $EndComp
 $Comp
-L GND #PWR089
+L GND #PWR099
 U 1 1 5AB969D7
 P 1950 1125
-F 0 "#PWR089" H 1950 875 50  0001 C CNN
+F 0 "#PWR099" H 1950 875 50  0001 C CNN
 F 1 "GND" H 1950 975 50  0000 C CNN
 F 2 "" H 1950 1125 50  0001 C CNN
@@
 Connection ~ 1950 775
 $Comp
-L R_Pack04 RN14
+L R_Pack04 RN702
 U 1 1 5AB97052
 P 1900 2625
-F 0 "RN14" V 1600 2625 50  0000 C CNN
+F 0 "RN702" V 1600 2625 50  0000 C CNN
 F 1 "51R" V 2100 2625 50  0000 C CNN
 F 2 "Resistor:0603_RN4" V 2175 2625 50  0001 C CNN
@@
 $EndComp
 $Comp
-L R_Pack04 RN15
+L R_Pack04 RN703
 U 1 1 5AB970C7
 P 1900 3400
-F 0 "RN15" V 1600 3400 50  0000 C CNN
+F 0 "RN703" V 1600 3400 50  0000 C CNN
 F 1 "51R" V 2100 3400 50  0000 C CNN
 F 2 "Resistor:0603_RN4" V 2175 3400 50  0001 C CNN
@@
 $EndComp
 $Comp
-L R_Pack04 RN16
+L R_Pack04 RN704
 U 1 1 5AB9723A
 P 1900 4175
-F 0 "RN16" V 1600 4175 50  0000 C CNN
+F 0 "RN704" V 1600 4175 50  0000 C CNN
 F 1 "51R" V 2100 4175 50  0000 C CNN
 F 2 "Resistor:0603_RN4" V 2175 4175 50  0001 C CNN
@@
 $EndComp
 $Comp
-L R_Pack04 RN17
+L R_Pack04 RN705
 U 1 1 5AB97385
 P 1900 4950
-F 0 "RN17" V 1600 4950 50  0000 C CNN
+F 0 "RN705" V 1600 4950 50  0000 C CNN
 F 1 "51R" V 2100 4950 50  0000 C CNN
 F 2 "Resistor:0603_RN4" V 2175 4950 50  0001 C CNN
@@
 $EndComp
 $Comp
-L R_Pack04 RN18
+L R_Pack04 RN706
 U 1 1 5AB984F2
 P 1900 5750
-F 0 "RN18" V 1600 5750 50  0000 C CNN
+F 0 "RN706" V 1600 5750 50  0000 C CNN
 F 1 "51R" V 2100 5750 50  0000 C CNN
 F 2 "Resistor:0603_RN4" V 2175 5750 50  0001 C CNN
@@
 $EndComp
 $Comp
-L R_Pack04 RN19
+L R_Pack04 RN707
 U 1 1 5AB984F8
 P 1900 6525
-F 0 "RN19" V 1600 6525 50  0000 C CNN
+F 0 "RN707" V 1600 6525 50  0000 C CNN
 F 1 "51R" V 2100 6525 50  0000 C CNN
 F 2 "Resistor:0603_RN4" V 2175 6525 50  0001 C CNN
@@
 $EndComp
 $Comp
-L R_Pack04 RN20
+L R_Pack04 RN708
 U 1 1 5AB984FE
 P 1900 7300
-F 0 "RN20" V 1600 7300 50  0000 C CNN
+F 0 "RN708" V 1600 7300 50  0000 C CNN
 F 1 "51R" V 2100 7300 50  0000 C CNN
 F 2 "Resistor:0603_RN4" V 2175 7300 50  0001 C CNN
@@
 LCD_B7
 $Comp
-L R_Pack04 RN13
+L R_Pack04 RN701
 U 1 1 5AB9F8D3
 P 1900 1875
-F 0 "RN13" V 1600 1875 50  0000 C CNN
+F 0 "RN701" V 1600 1875 50  0000 C CNN
 F 1 "51R" V 2100 1875 50  0000 C CNN
 F 2 "Resistor:0603_RN4" V 2175 1875 50  0001 C CNN
@@
 	1575 7400 1700 7400
 $Comp
-L TVS_8-Channel D6
+L TVS_8-Channel D701
 U 1 1 5ABA9419
 P 4350 2125
-F 0 "D6" H 4150 2675 60  0000 C CNN
+F 0 "D701" H 4150 2675 60  0000 C CNN
 F 1 "DT1240A-08LP3810" H 4350 1525 60  0000 C CNN
 F 2 "ESD:U-DFN3810-9" H 4100 1625 60  0001 C CNN
@@
 $EndComp
 $Comp
-L TVS_8-Channel D7
+L TVS_8-Channel D702
 U 1 1 5ABA97F4
 P 4350 3650
-F 0 "D7" H 4150 4200 60  0000 C CNN
+F 0 "D702" H 4150 4200 60  0000 C CNN
 F 1 "DT1240A-08LP3810" H 4350 3050 60  0000 C CNN
 F 2 "ESD:U-DFN3810-9" H 4100 3150 60  0001 C CNN
@@
 $EndComp
 $Comp
-L TVS_8-Channel D8
+L TVS_8-Channel D703
 U 1 1 5ABA98A3
 P 4350 5200
-F 0 "D8" H 4150 5750 60  0000 C CNN
+F 0 "D703" H 4150 5750 60  0000 C CNN
 F 1 "DT1240A-08LP3810" H 4350 4600 60  0000 C CNN
 F 2 "ESD:U-DFN3810-9" H 4100 4700 60  0001 C CNN
@@
 $EndComp
 $Comp
-L TVS_8-Channel D9
+L TVS_8-Channel D704
 U 1 1 5ABA9A40
 P 4350 6775
-F 0 "D9" H 4150 7325 60  0000 C CNN
+F 0 "D704" H 4150 7325 60  0000 C CNN
 F 1 "DT1240A-08LP3810" H 4350 6175 60  0000 C CNN
 F 2 "ESD:U-DFN3810-9" H 4100 6275 60  0001 C CNN
@@
 	3800 7175 3900 7175
 $Comp
-L GND #PWR090
+L GND #PWR0100
 U 1 1 5ABB29AB
 P 3875 2125
-F 0 "#PWR090" H 3875 1875 50  0001 C CNN
+F 0 "#PWR0100" H 3875 1875 50  0001 C CNN
 F 1 "GND" V 3875 1925 50  0000 C CNN
 F 2 "" H 3875 2125 50  0001 C CNN
@@
 	3875 2125 3900 2125
 $Comp
-L GND #PWR091
+L GND #PWR0101
 U 1 1 5ABB2CDD
 P 3875 3650
-F 0 "#PWR091" H 3875 3400 50  0001 C CNN
+F 0 "#PWR0101" H 3875 3400 50  0001 C CNN
 F 1 "GND" V 3875 3450 50  0000 C CNN
 F 2 "" H 3875 3650 50  0001 C CNN
@@
 $EndComp
 $Comp
-L GND #PWR092
+L GND #PWR0102
 U 1 1 5ABB3065
 P 3875 5200
-F 0 "#PWR092" H 3875 4950 50  0001 C CNN
+F 0 "#PWR0102" H 3875 4950 50  0001 C CNN
 F 1 "GND" V 3875 5000 50  0000 C CNN
 F 2 "" H 3875 5200 50  0001 C CNN
@@
 $EndComp
 $Comp
-L GND #PWR093
+L GND #PWR0103
 U 1 1 5ABB33CB
 P 3850 6775
-F 0 "#PWR093" H 3850 6525 50  0001 C CNN
+F 0 "#PWR0103" H 3850 6525 50  0001 C CNN
 F 1 "GND" V 3850 6575 50  0000 C CNN
 F 2 "" H 3850 6775 50  0001 C CNN
@@
 	3850 6775 3900 6775
 $Comp
-L Conn_01x06_Female J3
+L Conn_01x06_Female J702
 U 1 1 5ABC116D
 P 10400 3300
-F 0 "J3" H 10400 3600 50  0000 C CNN
+F 0 "J702" H 10400 3600 50  0000 C CNN
 F 1 "Conn_01x06_Female" H 10400 2900 50  0000 C CNN
 F 2 "Molex:52808-0671" H 10400 3300 50  0001 C CNN
@@
 $EndComp
 $Comp
-L TVS_8-Channel D10
+L TVS_8-Channel D705
 U 1 1 5ABC1710
 P 10125 2000
-F 0 "D10" H 9925 2550 60  0000 C CNN
+F 0 "D705" H 9925 2550 60  0000 C CNN
 F 1 "DT1240A-08LP3810" H 10125 1400 60  0000 C CNN
 F 2 "ESD:U-DFN3810-9" H 9875 1500 60  0001 C CNN
@@
 TFT_SCL
 $Comp
-L GND #PWR094
+L GND #PWR0104
 U 1 1 5ABC279B
 P 10150 3500
-F 0 "#PWR094" H 10150 3250 50  0001 C CNN
+F 0 "#PWR0104" H 10150 3250 50  0001 C CNN
 F 1 "GND" V 10150 3300 50  0000 C CNN
 F 2 "" H 10150 3500 50  0001 C CNN
@@
 Connection ~ 9600 2350
 $Comp
-L GND #PWR095
+L GND #PWR0105
 U 1 1 5ABC535D
 P 9600 2000
-F 0 "#PWR095" H 9600 1750 50  0001 C CNN
+F 0 "#PWR0105" H 9600 1750 50  0001 C CNN
 F 1 "GND" V 9600 1800 50  0000 C CNN
 F 2 "" H 9600 2000 50  0001 C CNN
@@
 	9600 2000 9675 2000
 $Comp
-L R_Pack04 RN21
+L R_Pack04 RN709
 U 1 1 5ABC6DD1
 P 7800 1850
-F 0 "RN21" V 7500 1850 50  0000 C CNN
+F 0 "RN709" V 7500 1850 50  0000 C CNN
 F 1 "51R" V 8000 1850 50  0000 C CNN
 F 2 "Resistor:0603_RN4" V 8075 1850 50  0001 C CNN
@@
 Text Notes 10300 7500 0    60   ~ 0
 By Jesse Spiessens
+NoConn ~ 6025 2125
+NoConn ~ 6025 1925
+NoConn ~ 6025 1825
+NoConn ~ 6025 1725
+NoConn ~ 6025 1625
+NoConn ~ 1700 1675
+NoConn ~ 2100 1675
+NoConn ~ 1700 2425
+NoConn ~ 2100 2425
+NoConn ~ 2100 2525
+NoConn ~ 2100 2625
+NoConn ~ 1700 2625
+NoConn ~ 1700 2525
+NoConn ~ 3900 2025
+NoConn ~ 3900 3350
+NoConn ~ 3900 3450
+NoConn ~ 3900 3550
 $EndSCHEMATC
