File: PCB/DSP board/Supply.sch (KiCad schematic (older format))
At the start: 39 parts, among them U4 MIC23050, U5 TPS2113A, U6 TPS61170, U7 ADP150

Commit message: Schematics + Footprints Rev.1
Ready to route.
Parts:
- C81, C83, C84, C87, C88, C90, C91, C92, C93, C94, C95, C96, C97: footprint (none) -> Capacitors_SMD:C_0603
- C82, C85, C89: footprint (none) -> Capacitors_SMD:C_0805
- C86: footprint (none) -> Capacitors_SMD:C_1206
- D2: footprint (none) -> Diodes_SMD:D_SOD-523
- D3, D4: footprint (none) -> Diodes_SMD:D_SMA
- D5: footprint (none) -> SOD:SOD-323F-2
- F1, R10, R3, R4, R5, R6, R7, R9: footprint (none) -> Resistors_SMD:R_0603
- L5, L6, L9: footprint (none) -> Inductors_SMD:L_0603
- L7, L8: footprint (none) -> Inductors_SMD:L_0805
- R8: footprint (none) -> Resistors_SMD:R_0805
- U4: footprint (none) -> Housings_DFN_QFN:DFN-8-1EP_2x2mm_Pitch0.5mm
- U5: footprint (none) -> Housings_DFN_QFN:DFN-8-1EP_3x3mm_Pitch0.65mm
- U6: footprint (none) -> Housings_DFN_QFN:DFN-6-1EP_2x2mm_Pitch0.65mm
- U7: footprint (none) -> Housings_SSOP:TSOP-5_1.65x3.05mm_Pitch0.95mm

Commit message: Schematics & PCB
Schematics update - ERC error fixing
PCB - setup & PCB outline
Parts:
- renumbered C81 to C601, C82 to C602, C83 to C603, C84 to C604, C85 to C605, C86 to C606, C87 to C607, C88 to C608, C89 to C609, C90 to C610, C91 to C611, C92 to C612, C93 to C613, C94 to C614, C95 to C615, C96 to C616, C97 to C617, D2 to D601, D3 to D602, D4 to D603, D5 to D604, F1 to F601, L5 to L601, L6 to L602, L7 to L603, L8 to L604, L9 to L605, R3 to R601, R4 to R602, R5 to R603, R6 to R604, R7 to R605, R8 to R606, R9 to R607, R10 to R608, U4 to U601, U5 to U602, U6 to U603, U7 to U604
