File: PCB/IO board/Audio Supplies.sch (KiCad schematic (older format))
At the start: 28 parts

Commit message: Schematics Rev 1.0
Parts:
- gave numbers to parts that had none: 27

Commit message: Component Placement - No pul-up
ALmost finished component placement expect for pull ups and low pass
filters for switches etc
Parts:
- C401, C404, C405, C407, C411, C412: footprint (none) -> Capacitors_SMD:C_0805
- C402, C403, C406, C408, C409: footprint (none) -> Capacitors_SMD:C_0603
- C410: footprint (none) -> Capacitors_SMD:C_1206
- D401, D402, D403: footprint (none) -> Diodes_SMD:D_SOD-123F
- L401: footprint (none) -> Inductors_SMD:L_0603
- L402: footprint (none) -> Inductors_SMD:L_0805
- R401, R403, R405: footprint (none) -> Resistors_SMD:R_0805
- R402, R404, R406, R407, R408: footprint (none) -> Resistors_SMD:R_0603
- U401: footprint (none) -> Housings_SOIC:SOIC-8_3.9x4.9mm_Pitch1.27mm
- U402: footprint (none) -> Housings_DFN_QFN:DFN-6-1EP_2x2mm_Pitch0.65mm
Changed lines of the file:
@@
 F 0 "U401" H 3325 1950 50  0000 L CNN
 F 1 "MCP6002-xSN" H 3325 1600 50  0000 L CNN
-F 2 "" H 3325 1800 50  0001 C CNN
+F 2 "Housings_SOIC:SOIC-8_3.9x4.9mm_Pitch1.27mm" H 3325 1800 50  0001 C CNN
 F 3 "" H 3325 1800 50  0001 C CNN
 	1    3325 1800
@@
 F 0 "U401" H 3325 2800 50  0000 L CNN
 F 1 "MCP6002-xSN" H 3325 2450 50  0000 L CNN
-F 2 "" H 3325 2650 50  0001 C CNN
+F 2 "Housings_SOIC:SOIC-8_3.9x4.9mm_Pitch1.27mm" H 3325 2650 50  0001 C CNN
 F 3 "" H 3325 2650 50  0001 C CNN
 	2    3325 2650
@@
 F 0 "R402" H 1950 2125 50  0000 C CNN
 F 1 "1k5" V 2100 2050 50  0000 C CNN
-F 2 "" V 2030 2050 50  0001 C CNN
+F 2 "Resistors_SMD:R_0603" V 2030 2050 50  0001 C CNN
 F 3 "" H 2100 2050 50  0001 C CNN
 	1    2100 2050
@@
 F 0 "R404" H 1950 2525 50  0000 C CNN
 F 1 "1k5" V 2100 2450 50  0000 C CNN
-F 2 "" V 2030 2450 50  0001 C CNN
+F 2 "Resistors_SMD:R_0603" V 2030 2450 50  0001 C CNN
 F 3 "" H 2100 2450 50  0001 C CNN
 	1    2100 2450
@@
 F 0 "C403" H 2385 2520 50  0000 L CNN
 F 1 "1uF" H 2385 2370 50  0000 L CNN
-F 2 "" H 2375 2450 50  0001 C CNN
+F 2 "Capacitors_SMD:C_0603" H 2375 2450 50  0001 C CNN
 F 3 "" H 2375 2450 50  0001 C CNN
 	1    2375 2450
@@
 F 0 "C402" V 2950 2000 50  0000 L CNN
 F 1 "100nF" V 2950 2250 50  0000 L CNN
-F 2 "" H 3000 2225 50  0001 C CNN
+F 2 "Capacitors_SMD:C_0603" H 3000 2225 50  0001 C CNN
 F 3 "" H 3000 2225 50  0001 C CNN
 	1    3000 2225
@@
 F 0 "C406" H 1860 4495 50  0000 L CNN
 F 1 "100nF" H 1860 4345 50  0000 L CNN
-F 2 "" H 1850 4425 50  0001 C CNN
+F 2 "Capacitors_SMD:C_0603" H 1850 4425 50  0001 C CNN
 F 3 "" H 1850 4425 50  0001 C CNN
 	1    1850 4425
@@
 F 0 "L401" V 2125 4250 50  0000 L CNN
 F 1 "1k 400mA" V 2125 3775 50  0000 L CNN
-F 2 "" V 1980 4225 50  0001 C CNN
+F 2 "Inductors_SMD:L_0603" V 1980 4225 50  0001 C CNN
 F 3 "" H 2050 4225 50  0001 C CNN
 	1    2050 4225
@@
 F 0 "C407" H 2260 4495 50  0000 L CNN
 F 1 "4.7uF" H 2260 4345 50  0000 L CNN
-F 2 "" H 2250 4425 50  0001 C CNN
+F 2 "Capacitors_SMD:C_0805" H 2250 4425 50  0001 C CNN
 F 3 "" H 2250 4425 50  0001 C CNN
 	1    2250 4425
@@
 F 0 "C408" H 2585 4495 50  0000 L CNN
 F 1 "100nF" H 2585 4345 50  0000 L CNN
-F 2 "" H 2575 4425 50  0001 C CNN
+F 2 "Capacitors_SMD:C_0603" H 2575 4425 50  0001 C CNN
 F 3 "" H 2575 4425 50  0001 C CNN
 	1    2575 4425
@@
 F 0 "U402" H 4275 4775 60  0000 C CNN
 F 1 "TPS61170" H 4275 3975 60  0000 C CNN
-F 2 "" H 3975 4125 60  0001 C CNN
+F 2 "Housings_DFN_QFN:DFN-6-1EP_2x2mm_Pitch0.65mm" H 3975 4125 60  0001 C CNN
 F 3 "" H 3975 4125 60  0001 C CNN
 	1    4275 4425
@@
 F 0 "L402" H 3200 4300 50  0000 C CNN
 F 1 "15uH" H 3000 4550 50  0000 C CNN
-F 2 "" H 3100 4425 50  0001 C CNN
+F 2 "Inductors_SMD:L_0805" H 3100 4425 50  0001 C CNN
 F 3 "" H 3100 4425 50  0001 C CNN
 	1    3100 4425
@@
 F 0 "C410" H 2875 4800 50  0000 L CNN
 F 1 "1uF" H 2925 4975 50  0000 L CNN
-F 2 "" H 3100 4875 50  0001 C CNN
+F 2 "Capacitors_SMD:C_1206" H 3100 4875 50  0001 C CNN
 F 3 "" H 3100 4875 50  0001 C CNN
 	1    3100 4875
@@
 F 0 "D401" V 3775 4775 50  0000 C CNN
 F 1 "2SS100L-W" V 3550 5125 50  0000 C CNN
-F 2 "" H 3675 4875 50  0001 C CNN
+F 2 "Diodes_SMD:D_SOD-123F" H 3675 4875 50  0001 C CNN
 F 3 "" H 3675 4875 50  0001 C CNN
 	1    3675 4875
@@
 F 0 "D402" H 3275 5025 50  0000 C CNN
 F 1 "2SS100L-W" H 3400 5175 50  0000 C CNN
-F 2 "" H 3425 5075 50  0001 C CNN
+F 2 "Diodes_SMD:D_SOD-123F" H 3425 5075 50  0001 C CNN
 F 3 "" H 3425 5075 50  0001 C CNN
 	1    3425 5075
@@
 F 0 "D403" V 3200 5175 50  0000 C CNN
 F 1 "2SS100L-W" V 3000 5025 50  0000 C CNN
-F 2 "" H 3100 5275 50  0001 C CNN
+F 2 "Diodes_SMD:D_SOD-123F" H 3100 5275 50  0001 C CNN
 F 3 "" H 3100 5275 50  0001 C CNN
 	1    3100 5275
@@
 F 0 "C411" H 3475 5350 50  0000 L CNN
 F 1 "4.7uF" H 3425 5200 50  0000 L CNN
-F 2 "" H 3675 5275 50  0001 C CNN
+F 2 "Capacitors_SMD:C_0805" H 3675 5275 50  0001 C CNN
 F 3 "" H 3675 5275 50  0001 C CNN
 	1    3675 5275
@@
 F 0 "C412" H 3725 5600 50  0000 L CNN
 F 1 "4.7uF" H 3725 5750 50  0000 L CNN
-F 2 "" H 3675 5675 50  0001 C CNN
+F 2 "Capacitors_SMD:C_0805" H 3675 5675 50  0001 C CNN
 F 3 "" H 3675 5675 50  0001 C CNN
 	1    3675 5675
@@
 F 0 "R406" H 5025 4075 50  0000 C CNN
 F 1 "470k" V 4875 4000 50  0000 C CNN
-F 2 "" V 4805 4000 50  0001 C CNN
+F 2 "Resistors_SMD:R_0603" V 4805 4000 50  0001 C CNN
 F 3 "" H 4875 4000 50  0001 C CNN
 	1    4875 4000
@@
 F 0 "R407" V 5025 4225 50  0000 C CNN
 F 1 "12k" V 5100 4225 50  0000 C CNN
-F 2 "" V 5030 4225 50  0001 C CNN
+F 2 "Resistors_SMD:R_0603" V 5030 4225 50  0001 C CNN
 F 3 "" H 5100 4225 50  0001 C CNN
 	1    5100 4225
@@
 F 0 "R408" V 5180 4425 50  0000 C CNN
 F 1 "12k" V 5100 4425 50  0000 C CNN
-F 2 "" V 5030 4425 50  0001 C CNN
+F 2 "Resistors_SMD:R_0603" V 5030 4425 50  0001 C CNN
 F 3 "" H 5100 4425 50  0001 C CNN
 	1    5100 4425
@@
 F 0 "C409" H 5360 4695 50  0000 L CNN
 F 1 "10nF" H 5360 4545 50  0000 L CNN
-F 2 "" H 5350 4625 50  0001 C CNN
+F 2 "Capacitors_SMD:C_0603" H 5350 4625 50  0001 C CNN
 F 3 "" H 5350 4625 50  0001 C CNN
 	1    5350 4625
@@
 F 0 "R401" V 7130 1375 50  0000 C CNN
 F 1 "10R" V 7050 1375 50  0000 C CNN
-F 2 "" V 6980 1375 50  0001 C CNN
+F 2 "Resistors_SMD:R_0805" V 6980 1375 50  0001 C CNN
 F 3 "" H 7050 1375 50  0001 C CNN
 	1    7050 1375
@@
 F 0 "C401" H 7310 1645 50  0000 L CNN
 F 1 "22uF" H 7310 1495 50  0000 L CNN
-F 2 "" H 7300 1575 50  0001 C CNN
+F 2 "Capacitors_SMD:C_0805" H 7300 1575 50  0001 C CNN
 F 3 "" H 7300 1575 50  0001 C CNN
 	1    7300 1575
@@
 F 0 "R403" V 7130 2375 50  0000 C CNN
 F 1 "10R" V 7050 2375 50  0000 C CNN
-F 2 "" V 6980 2375 50  0001 C CNN
+F 2 "Resistors_SMD:R_0805" V 6980 2375 50  0001 C CNN
 F 3 "" H 7050 2375 50  0001 C CNN
 	1    7050 2375
@@
 F 0 "C404" H 7310 2645 50  0000 L CNN
 F 1 "22uF" H 7310 2495 50  0000 L CNN
-F 2 "" H 7300 2575 50  0001 C CNN
+F 2 "Capacitors_SMD:C_0805" H 7300 2575 50  0001 C CNN
 F 3 "" H 7300 2575 50  0001 C CNN
 	1    7300 2575
@@
 F 0 "R405" V 7130 3375 50  0000 C CNN
 F 1 "10R" V 7050 3375 50  0000 C CNN
-F 2 "" V 6980 3375 50  0001 C CNN
+F 2 "Resistors_SMD:R_0805" V 6980 3375 50  0001 C CNN
 F 3 "" H 7050 3375 50  0001 C CNN
 	1    7050 3375
@@
 F 0 "C405" H 7310 3645 50  0000 L CNN
 F 1 "22uF" H 7310 3495 50  0000 L CNN
-F 2 "" H 7300 3575 50  0001 C CNN
+F 2 "Capacitors_SMD:C_0805" H 7300 3575 50  0001 C CNN
 F 3 "" H 7300 3575 50  0001 C CNN
 	1    7300 3575
