File: PCB/IO board/IO.sch (KiCad schematic (older format))
At the start: 45 parts

Commit message: Schematics Rev 1.0
Parts:
- gave numbers to parts that had none: 45

Commit message: Component Placement - No pul-up
ALmost finished component placement expect for pull ups and low pass
filters for switches etc
Parts:
- C701, C702, C703, C704, C705, C706, C707, C708, C709, C710, C711, C712: footprint (none) -> Capacitors_SMD:C_0603
- R701, R702, R703, R704, R705, R706, R707, R708, R709, R710, R711, R712, R713, R714, R715, R716, R717, R718, R719, R720, R721, R722, R723, R724, R725, R726, R727: footprint (none) -> Resistors_SMD:R_0603
- S701, S702, S703: footprint (none) -> ELECTROMECH:PEL12D-4xxxS
- SW701, SW702, SW703: footprint (none) -> ELECTROMECH:PS1024A

Commit message: PCB Backup
Parts:
- added R728, R729, R730: 12k, Resistors_SMD:R_0603, symbol R
Connections:
- net ENCODER_1_SW: now also R728.1; no longer R719.2, S701.4 (S)
- net ENCODER_2_SW: now also R729.1; no longer R720.2, S702.4 (S)
- net ENCODER_3_SW: now also R730.1; no longer R721.2, S703.4 (S)
- new net: R719.2, R728.2, S701.4 (S)
- new net: R720.2, R729.2, S702.4 (S)
- new net: R721.2, R730.2, S703.4 (S)
Other:
- moved on the sheet: C707, C708, C709, R719, R720, R721
