File: PCB/IO board/ESP.sch (KiCad schematic (older format))
At the start: 15 parts, among them J801 Conn_01x06_Male, U801 ESP32S, U802 ESP32

Commit message: Component Placement - No pul-up
ALmost finished component placement expect for pull ups and low pass
filters for switches etc
Parts:
- C801, C802, C803, C804, C805: footprint (none) -> Capacitors_SMD:C_0603
- J801: footprint (none) -> Pin_Headers:Pin_Header_Straight_1x06_Pitch2.54mm_SMD_Pin1Right
- L801: footprint (none) -> Inductors_SMD:L_0603_HandSoldering
- R801, R802, R803, R804: footprint (none) -> Resistors_SMD:R_0603
- S801, S802: footprint (none) -> Switch:FSM4JSMATR
- U801: footprint (none) -> WIFI:ESP32S
- U802: footprint (none) -> WIFI:ESP32
Changed lines of the file:
@@
 F 0 "U801" H 3750 3000 60  0000 C CNN
 F 1 "ESP32S" H 3750 850 60  0000 C CNN
-F 2 "" H 3650 2400 60  0001 C CNN
+F 2 "WIFI:ESP32S" H 3650 2400 60  0001 C CNN
 F 3 "" H 3650 2400 60  0001 C CNN
 	1    3750 2000
@@
 $EndComp
 $Comp
-L GND #PWR0129
+L GND #PWR0130
 U 1 1 5AE61B01
 P 3000 1150
-F 0 "#PWR0129" H 3000 900 50  0001 C CNN
+F 0 "#PWR0130" H 3000 900 50  0001 C CNN
 F 1 "GND" V 2975 975 50  0000 C CNN
 F 2 "" H 3000 1150 50  0001 C CNN
@@
 $EndComp
 $Comp
-L +3V3 #PWR0130
+L +3V3 #PWR0131
 U 1 1 5AE61B07
 P 1150 1250
-F 0 "#PWR0130" H 1150 1100 50  0001 C CNN
+F 0 "#PWR0131" H 1150 1100 50  0001 C CNN
 F 1 "+3V3" H 1150 1390 50  0000 C CNN
 F 2 "" H 1150 1250 50  0001 C CNN
@@
 F 0 "L801" V 1525 1300 50  0000 L CNN
 F 1 "220R" V 1375 1025 50  0000 L CNN
-F 2 "" V 1380 1250 50  0001 C CNN
+F 2 "Inductors_SMD:L_0603_HandSoldering" V 1380 1250 50  0001 C CNN
 F 3 "" H 1450 1250 50  0001 C CNN
 	1    1450 1250
@@
 F 0 "C801" H 1260 1520 50  0000 L CNN
 F 1 "10nF" H 1260 1370 50  0000 L CNN
-F 2 "" H 1250 1450 50  0001 C CNN
+F 2 "Capacitors_SMD:C_0603" H 1250 1450 50  0001 C CNN
 F 3 "" H 1250 1450 50  0001 C CNN
 	1    1250 1450
@@
 F 0 "C802" H 1760 1520 50  0000 L CNN
 F 1 "1uF" H 1760 1370 50  0000 L CNN
-F 2 "" H 1750 1450 50  0001 C CNN
+F 2 "Capacitors_SMD:C_0603" H 1750 1450 50  0001 C CNN
 F 3 "" H 1750 1450 50  0001 C CNN
 	1    1750 1450
@@
 F 0 "C803" H 2060 1520 50  0000 L CNN
 F 1 "10nF" H 2060 1370 50  0000 L CNN
-F 2 "" H 2050 1450 50  0001 C CNN
+F 2 "Capacitors_SMD:C_0603" H 2050 1450 50  0001 C CNN
 F 3 "" H 2050 1450 50  0001 C CNN
 	1    2050 1450
@@
 $EndComp
 $Comp
-L GND #PWR0131
+L GND #PWR0132
 U 1 1 5AE61B29
 P 1250 1650
-F 0 "#PWR0131" H 1250 1400 50  0001 C CNN
+F 0 "#PWR0132" H 1250 1400 50  0001 C CNN
 F 1 "GND" H 1250 1500 50  0000 C CNN
 F 2 "" H 1250 1650 50  0001 C CNN
@@
 $EndComp
 $Comp
-L GND #PWR0132
+L GND #PWR0133
 U 1 1 5AE61B2F
 P 1750 1650
-F 0 "#PWR0132" H 1750 1400 50  0001 C CNN
+F 0 "#PWR0133" H 1750 1400 50  0001 C CNN
 F 1 "GND" H 1750 1500 50  0000 C CNN
 F 2 "" H 1750 1650 50  0001 C CNN
@@
 $EndComp
 $Comp
-L GND #PWR0133
+L GND #PWR0134
 U 1 1 5AE61B35
 P 2050 1650
-F 0 "#PWR0133" H 2050 1400 50  0001 C CNN
+F 0 "#PWR0134" H 2050 1400 50  0001 C CNN
 F 1 "GND" H 2050 1500 50  0000 C CNN
 F 2 "" H 2050 1650 50  0001 C CNN
@@
 F 0 "S801" V 2125 2125 60  0000 C CNN
 F 1 "Switch_SPST_4Pin" V 1675 2125 60  0000 C CNN
-F 2 "" H 1700 2225 60  0001 C CNN
+F 2 "Switch:FSM4JSMATR" H 1700 2225 60  0001 C CNN
 F 3 "" H 1700 2225 60  0001 C CNN
 	1    1900 2125
@@
 F 0 "R801" V 2630 1350 50  0000 C CNN
 F 1 "12k" V 2550 1350 50  0000 C CNN
-F 2 "" V 2480 1350 50  0001 C CNN
+F 2 "Resistors_SMD:R_0603" V 2480 1350 50  0001 C CNN
 F 3 "" H 2550 1350 50  0001 C CNN
 	1    2550 1350
@@
 F 0 "C804" H 2810 1620 50  0000 L CNN
 F 1 "10nF" H 2810 1470 50  0000 L CNN
-F 2 "" H 2800 1550 50  0001 C CNN
+F 2 "Capacitors_SMD:C_0603" H 2800 1550 50  0001 C CNN
 F 3 "" H 2800 1550 50  0001 C CNN
 	1    2800 1550
@@
 $EndComp
 $Comp
-L GND #PWR0134
+L GND #PWR0135
 U 1 1 5AE61B55
 P 2800 1750
-F 0 "#PWR0134" H 2800 1500 50  0001 C CNN
+F 0 "#PWR0135" H 2800 1500 50  0001 C CNN
 F 1 "GND" H 2800 1600 50  0000 C CNN
 F 2 "" H 2800 1750 50  0001 C CNN
@@
 $EndComp
 $Comp
-L GND #PWR0135
+L GND #PWR0136
 U 1 1 5AE61B5B
 P 2300 2425
-F 0 "#PWR0135" H 2300 2175 50  0001 C CNN
+F 0 "#PWR0136" H 2300 2175 50  0001 C CNN
 F 1 "GND" H 2300 2275 50  0000 C CNN
 F 2 "" H 2300 2425 50  0001 C CNN
@@
 F 0 "R802" V 1480 1975 50  0000 C CNN
 F 1 "12k" V 1400 1975 50  0000 C CNN
-F 2 "" V 1330 1975 50  0001 C CNN
+F 2 "Resistors_SMD:R_0603" V 1330 1975 50  0001 C CNN
 F 3 "" H 1400 1975 50  0001 C CNN
 	1    1400 1975
@@
 $EndComp
 $Comp
-L +3V3 #PWR0136
+L +3V3 #PWR0137
 U 1 1 5AE61B68
 P 1150 1975
-F 0 "#PWR0136" H 1150 1825 50  0001 C CNN
+F 0 "#PWR0137" H 1150 1825 50  0001 C CNN
 F 1 "+3V3" V 1175 2175 50  0000 C CNN
 F 2 "" H 1150 1975 50  0001 C CNN
@@
 F 0 "R804" V 5630 2450 50  0000 C CNN
 F 1 "12k" V 5550 2450 50  0000 C CNN
-F 2 "" V 5480 2450 50  0001 C CNN
+F 2 "Resistors_SMD:R_0603" V 5480 2450 50  0001 C CNN
 F 3 "" H 5550 2450 50  0001 C CNN
 	1    5550 2450
@@
 F 0 "C805" H 5300 2725 50  0000 L CNN
 F 1 "10nF" H 5100 2575 50  0000 L CNN
-F 2 "" H 5300 2650 50  0001 C CNN
+F 2 "Capacitors_SMD:C_0603" H 5300 2650 50  0001 C CNN
 F 3 "" H 5300 2650 50  0001 C CNN
 	1    5300 2650
@@
 $EndComp
 $Comp
-L GND #PWR0137
+L GND #PWR0138
 U 1 1 5AE61B7C
 P 5300 2850
-F 0 "#PWR0137" H 5300 2600 50  0001 C CNN
+F 0 "#PWR0138" H 5300 2600 50  0001 C CNN
 F 1 "GND" H 5300 2700 50  0000 C CNN
 F 2 "" H 5300 2850 50  0001 C CNN
@@
 F 0 "S802" V 6325 2600 60  0000 C CNN
 F 1 "Switch_SPST_4Pin" V 5875 2625 60  0000 C CNN
-F 2 "" H 5900 2700 60  0001 C CNN
+F 2 "Switch:FSM4JSMATR" H 5900 2700 60  0001 C CNN
 F 3 "" H 5900 2700 60  0001 C CNN
 	1    6100 2600
@@
 $EndComp
 $Comp
-L GND #PWR0138
+L GND #PWR0139
 U 1 1 5AE61B89
 P 5700 2900
-F 0 "#PWR0138" H 5700 2650 50  0001 C CNN
+F 0 "#PWR0139" H 5700 2650 50  0001 C CNN
 F 1 "GND" H 5700 2750 50  0000 C CNN
 F 2 "" H 5700 2900 50  0001 C CNN
@@
 F 0 "R803" H 6600 2125 50  0000 C CNN
 F 1 "12k" V 6450 2200 50  0000 C CNN
-F 2 "" V 6380 2200 50  0001 C CNN
+F 2 "Resistors_SMD:R_0603" V 6380 2200 50  0001 C CNN
 F 3 "" H 6450 2200 50  0001 C CNN
 	1    6450 2200
@@
 $EndComp
 $Comp
-L +3V3 #PWR0139
+L +3V3 #PWR0140
 U 1 1 5AE61B96
 P 6450 1950
-F 0 "#PWR0139" H 6450 1800 50  0001 C CNN
+F 0 "#PWR0140" H 6450 1800 50  0001 C CNN
 F 1 "+3V3" H 6475 2100 50  0000 C CNN
 F 2 "" H 6450 1950 50  0001 C CNN
@@
 BLUE_3
 $Comp
-L GND #PWR0140
+L GND #PWR0141
 U 1 1 5AE61BA2
 P 4500 1150
-F 0 "#PWR0140" H 4500 900 50  0001 C CNN
+F 0 "#PWR0141" H 4500 900 50  0001 C CNN
 F 1 "GND" V 4525 975 50  0000 C CNN
 F 2 "" H 4500 1150 50  0001 C CNN
@@
 $EndComp
 $Comp
-L GND #PWR0141
+L GND #PWR0142
 U 1 1 5AE61BA8
 P 3075 2550
-F 0 "#PWR0141" H 3075 2300 50  0001 C CNN
+F 0 "#PWR0142" H 3075 2300 50  0001 C CNN
 F 1 "GND" V 3075 2350 50  0000 C CNN
 F 2 "" H 3075 2550 50  0001 C CNN
@@
 F 0 "J801" H 6250 1300 50  0000 C CNN
 F 1 "Conn_01x06_Male" H 6250 600 50  0000 C CNN
-F 2 "" H 6250 1000 50  0001 C CNN
+F 2 "Pin_Headers:Pin_Header_Straight_1x06_Pitch2.54mm_SMD_Pin1Right" H 6250 1000 50  0001 C CNN
 F 3 "" H 6250 1000 50  0001 C CNN
 	1    6250 1000
@@
 $EndComp
 $Comp
-L GND #PWR0142
+L GND #PWR0143
 U 1 1 5AE61BB5
 P 6025 800
-F 0 "#PWR0142" H 6025 550 50  0001 C CNN
+F 0 "#PWR0143" H 6025 550 50  0001 C CNN
 F 1 "GND" V 6000 625 50  0000 C CNN
 F 2 "" H 6025 800 50  0001 C CNN
@@
 BLUE_3
 $Comp
-L GND #PWR0143
+L GND #PWR0144
 U 1 1 5AE639B0
 P 3075 5450
-F 0 "#PWR0143" H 3075 5200 50  0001 C CNN
+F 0 "#PWR0144" H 3075 5200 50  0001 C CNN
 F 1 "GND" V 3075 5250 50  0000 C CNN
 F 2 "" H 3075 5450 50  0001 C CNN
@@
 	4400 5450 4500 5450
 $Comp
-L GND #PWR0144
+L GND #PWR0145
 U 1 1 5AE65441
 P 4500 4150
-F 0 "#PWR0144" H 4500 3900 50  0001 C CNN
+F 0 "#PWR0145" H 4500 3900 50  0001 C CNN
 F 1 "GND" V 4525 3975 50  0000 C CNN
 F 2 "" H 4500 4150 50  0001 C CNN
@@
 $EndComp
 $Comp
-L GND #PWR0145
+L GND #PWR0146
 U 1 1 5AE65985
 P 4425 4750
-F 0 "#PWR0145" H 4425 4500 50  0001 C CNN
+F 0 "#PWR0146" H 4425 4500 50  0001 C CNN
 F 1 "GND" V 4450 4575 50  0000 C CNN
 F 2 "" H 4425 4750 50  0001 C CNN
@@
 F 0 "U802" H 3750 6000 60  0000 C CNN
 F 1 "ESP32" H 3750 3850 60  0000 C CNN
-F 2 "" H 3650 5400 60  0001 C CNN
+F 2 "WIFI:ESP32" H 3650 5400 60  0001 C CNN
 F 3 "" H 3650 5400 60  0001 C CNN
 	1    3750 5000
@@
 NoConn ~ 1650 2275
 $Comp
-L PWR_FLAG #FLG0146
+L PWR_FLAG #FLG0147
 U 1 1 5AEA116E
 P 2050 1150
-F 0 "#FLG0146" H 2050 1225 50  0001 C CNN
+F 0 "#FLG0147" H 2050 1225 50  0001 C CNN
 F 1 "PWR_FLAG" H 2050 1300 50  0000 C CNN
 F 2 "" H 2050 1150 50  0001 C CNN

Commit message: PCB Backup
Connections:
- net +3V3: now also R802.1; no longer R802.2
- net BLUE_1: now also U801.33 (GPIO21), U802.33 (GPIO21); no longer U801.10 (GPIO25), U802.9 (GPIO25)
- net BLUE_2: now also U801.17 (GPIO9), U802.16 (GPIO9); no longer U801.12 (GPIO27), U802.11 (GPIO27)
- net ORANGE_1: now also U801.31 (GPIO19), U802.31 (GPIO19); no longer U801.11 (GPIO26), U802.10 (GPIO26)
- net ORANGE_2: now also U801.16 (GPIO13), U802.15 (GPIO13); no longer U801.13 (GPIO14), U802.12 (GPIO14)
- net ORANGE_3: now also U801.13 (GPIO14), U802.12 (GPIO14); no longer U801.16 (GPIO13), U802.15 (GPIO13)
- net Phantom: now also U801.12 (GPIO27), U802.11 (GPIO27); no longer U801.29 (GPIO5), U802.29 (GPIO5)
- net Phantom_1: now also U801.11 (GPIO26), U802.10 (GPIO26); no longer U801.31 (GPIO19), U802.31 (GPIO19)
- net Phantom_2: now also U801.10 (GPIO25), U802.9 (GPIO25); no longer U801.30 (GPIO18), U802.30 (GPIO18)
- net at S801.3: no longer R802.1
- net at R801.2, S801.4: now also R802.2
- no-connect marks 44 -> 45
Other:
- moved on the sheet: R802, S801

Commit message: IO board Rev 1.0 RC-1
Board for inspection by Supervisor
Connections:
- net ENCODER_1_A: now also J801.5 (Pin_5); no longer J801.4 (Pin_4)
- net ENCODER_1_B: now also J801.4 (Pin_4); no longer J801.5 (Pin_5)
Changed lines of the file:
@@
 Text GLabel 5950 1300 0    60   Input ~ 0
 ENCODER_1_SW
+Text GLabel 5950 1100 0    60   Input ~ 0
+ENCODER_1_B
 Text GLabel 5950 1200 0    60   Input ~ 0
-ENCODER_1_B
-Text GLabel 5950 1100 0    60   Input ~ 0
 ENCODER_1_A
 Wire Wire Line
