File: PCB/IO board/_autosave-Audio board.kicad_pcb (KiCad board)
At the start: 2 copper layers, 150 x 150 mm, 227 parts, among them J101 Screen_Standoff, J102 Screen_Standoff, J103 Standoff_MaGee, J104 Screen_Standoff, J105 Screen_Standoff, J301 6.3mm TRS, J501 Conn_01x02, J601 Jack-DC, J602 TEST_1P, J801 Conn_01x06_Male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

Commit message: IO board Rev 1.0 RC-1
Board for inspection by Supervisor
Parts:
- added G***: LOGO, Graphics:Logo_IO, F.Cu at (84.2, 67.0)
Other:
- board text added: "Aellö"
- board text added: "Rev 1.0"
- board text added: "by Jesse Spiessens"
